File: Overall schematic/overall scematic/digital_sensor.kicad_sch (KiCad schematic)
At the start: 0 parts

Commit message: Add files via upload
Parts:
- added U1: SHT4x, Sensor_Humidity:Sensirion_DFN-4_1.5x1.5mm_P0.8mm_SHT4x_NoCentralPad, symbol Sensor_Humidity:SHT4x
Connections:
- new net GND: U1.4 (VSS)
- new net SCL: U1.2 (SCL)
- new net SDA: U1.1 (SDA)
- new net VCC: U1.3 (VDD)
Changed lines of the file:
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@@
 (kicad_sch (version 20230121) (generator eeschema)
   (paper "A4")
+  (wire (pts (xy 121.92 95.25) (xy 121.92 100.33))
+    (stroke (width 0) (type default))
+  )
+  (wire (pts (xy 104.14 85.09) (xy 111.76 85.09))
+    (stroke (width 0) (type default))
+  )
+  (wire (pts (xy 104.14 90.17) (xy 111.76 90.17))
+    (stroke (width 0) (type default))
+  )
+  (wire (pts (xy 121.92 74.93) (xy 121.92 80.01))
+    (stroke (width 0) (type default))
+  )
+  (global_label "SCL" (shape output) (at 104.14 85.09 180) (fields_autoplaced)
+    (effects (font (size 1.27 1.27)) (justify right))
+    (property "Intersheetrefs" "${INTERSHEET_REFS}" (at 97.7266 85.09 0)
+      (effects (font (size 1.27 1.27)) (justify right) hide)
+    )
+  )
+  (global_label "SDA" (shape output) (at 104.14 90.17 180) (fields_autoplaced)
+    (effects (font (size 1.27 1.27)) (justify right))
+    (property "Intersheetrefs" "${INTERSHEET_REFS}" (at 97.6661 90.17 0)
+      (effects (font (size 1.27 1.27)) (justify right) hide)
+    )
+  )
+  (symbol (lib_id "power:VCC") (at 121.92 74.93 0) (unit 1)
+    (in_bom yes) (on_board yes) (dnp no) (fields_autoplaced)
+    (property "Reference" "#PWR02" (at 121.92 78.74 0)
+      (effects (font (size 1.27 1.27)) hide)
+    )
+    (property "Value" "VCC" (at 121.92 71.12 0)
+      (effects (font (size 1.27 1.27)))
+    )
+    (property "Footprint" "" (at 121.92 74.93 0)
+      (effects (font (size 1.27 1.27)) hide)
+    )
+    (property "Datasheet" "" (at 121.92 74.93 0)
+      (effects (font (size 1.27 1.27)) hide)
+    )
+    (pin "1")
+    (instances
+      (project "overall scematic"
+        (path "/9230863d-68c5-4e85-a5d4-0f54ecfbae5b/5eab94a0-95fb-4405-9961-390291429e6b"
+          (reference "#PWR02") (unit 1)
+        )
+      )
+    )
+  )
+  (symbol (lib_id "Sensor_Humidity:SHT4x") (at 119.38 87.63 0) (unit 1)
+    (in_bom yes) (on_board yes) (dnp no) (fields_autoplaced)
+    (property "Reference" "U1" (at 125.73 86.995 0)
+      (effects (font (size 1.27 1.27)) (justify left))
+    )
+    (property "Value" "SHT4x" (at 125.73 89.535 0)
+      (effects (font (size 1.27 1.27)) (justify left))
+    )
+    (property "Footprint" "Sensor_Humidity:Sensirion_DFN-4_1.5x1.5mm_P0.8mm_SHT4x_NoCentralPad" (at 123.19 93.98 0)
+      (effects (font (size 1.27 1.27)) (justify left) hide)
+    )
+    (property "Datasheet" "https://sensirion.com/media/documents/33FD6951/624C4357/Datasheet_SHT4x.pdf" (at 123.19 96.52 0)
+      (effects (font (size 1.27 1.27)) (justify left) hide)
+    )
+    (pin "1")
+    (pin "2")
+    (pin "3")
+    (pin "4")
+    (instances
+      (project "overall scematic"
+        (path "/9230863d-68c5-4e85-a5d4-0f54ecfbae5b/5eab94a0-95fb-4405-9961-390291429e6b"
+          (reference "U1") (unit 1)
+        )
+      )
+    )
+  )
+  (symbol (lib_id "power:GND") (at 121.92 100.33 0) (unit 1)
+    (in_bom yes) (on_board yes) (dnp no) (fields_autoplaced)
+    (property "Reference" "#PWR01" (at 121.92 106.68 0)
+      (effects (font (size 1.27 1.27)) hide)
+    )
+    (property "Value" "GND" (at 121.92 105.41 0)
+      (effects (font (size 1.27 1.27)))
+    )
+    (property "Footprint" "" (at 121.92 100.33 0)
+      (effects (font (size 1.27 1.27)) hide)
+    )
+    (property "Datasheet" "" (at 121.92 100.33 0)
+      (effects (font (size 1.27 1.27)) hide)
+    )
+    (pin "1")
+    (instances
+      (project "overall scematic"
+        (path "/9230863d-68c5-4e85-a5d4-0f54ecfbae5b/5eab94a0-95fb-4405-9961-390291429e6b"
+          (reference "#PWR01") (unit 1)
+        )
+      )
+    )
+  )
 )

Commit message: updated schematic
Connections:
- net VCC renamed 3v3
Changed lines of the file:
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@@
     (stroke (width 0) (type default))
   )
-  (global_label "SCL" (shape output) (at 104.14 85.09 180) (fields_autoplaced)
+  (hierarchical_label "SDA" (shape input) (at 104.14 90.17 180) (fields_autoplaced)
     (effects (font (size 1.27 1.27)) (justify right))
-    (property "Intersheetrefs" "${INTERSHEET_REFS}" (at 97.7266 85.09 0)
-      (effects (font (size 1.27 1.27)) (justify right) hide)
-    )
   )
-  (global_label "SDA" (shape output) (at 104.14 90.17 180) (fields_autoplaced)
+  (hierarchical_label "SCL" (shape input) (at 104.14 85.09 180) (fields_autoplaced)
     (effects (font (size 1.27 1.27)) (justify right))
-    (property "Intersheetrefs" "${INTERSHEET_REFS}" (at 97.6661 90.17 0)
-      (effects (font (size 1.27 1.27)) (justify right) hide)
-    )
   )
-  (symbol (lib_id "power:VCC") (at 121.92 74.93 0) (unit 1)
-    (in_bom yes) (on_board yes) (dnp no) (fields_autoplaced)
-    (property "Reference" "#PWR02" (at 121.92 78.74 0)
-      (effects (font (size 1.27 1.27)) hide)
-    )
-    (property "Value" "VCC" (at 121.92 71.12 0)
-      (effects (font (size 1.27 1.27)))
-    )
-    (property "Footprint" "" (at 121.92 74.93 0)
-      (effects (font (size 1.27 1.27)) hide)
-    )
-    (property "Datasheet" "" (at 121.92 74.93 0)
-      (effects (font (size 1.27 1.27)) hide)
-    )
-    (pin "1")
-    (instances
-      (project "overall scematic"
-        (path "/9230863d-68c5-4e85-a5d4-0f54ecfbae5b/5eab94a0-95fb-4405-9961-390291429e6b"
-          (reference "#PWR02") (unit 1)
-        )
-      )
-    )
+  (hierarchical_label "3v3" (shape input) (at 121.92 74.93 90) (fields_autoplaced)
+    (effects (font (size 1.27 1.27)) (justify left))
   )
   (symbol (lib_id "Sensor_Humidity:SHT4x") (at 119.38 87.63 0) (unit 1)
