File: Overall schematic/overall scematic/overall scematic.kicad_sch (KiCad schematic)
At the start: 0 parts

Commit message: updated interface
Other:
- added sheet Micro controller pin outs (micro controlter interface.kicad_sch)
- title: (none) -> overall schematic
Changed lines of the file:
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@@
 (kicad_sch (version 20230121) (generator eeschema)
   (paper "A4")
+  (title_block
+    (title "overall schematic")
+    (date "2023-03-10")
+    (rev "version1")
+  )
   (sheet (at 25.4 60.96) (size 54.61 17.78) (fields_autoplaced)
     (stroke (width 0.1524) (type solid))
@@
       )
     )
+  )
+  (sheet (at 127 66.04) (size 67.31 31.75) (fields_autoplaced)
+    (stroke (width 0.1524) (type solid))
+    (fill (color 0 0 0 0.0000))
+    (property "Sheetname" "Micro controller pin outs" (at 127 65.3284 0)
+      (effects (font (size 1.27 1.27)) (justify left bottom))
+    )
+    (property "Sheetfile" "micro controlter interface.kicad_sch" (at 127 98.3746 0)
+      (effects (font (size 1.27 1.27)) (justify left top))
+    )
+    (instances
+      (project "overall scematic"
+        (path "/9230863d-68c5-4e85-a5d4-0f54ecfbae5b" (page "7"))
+      )
+    )

Commit message: update kicad
Other:
- removed sheet Memory element
Changed lines of the file:
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@@
-    )
-  )
-  (sheet (at 25.4 24.13) (size 53.34 25.4) (fields_autoplaced)
-    (stroke (width 0.1524) (type solid))
-    (fill (color 0 0 0 0.0000))
-    (property "Sheetname" "Memory element" (at 25.4 23.4184 0)
-      (effects (font (size 1.27 1.27)) (justify left bottom))
-    )
-    (property "Sheetfile" "memory.kicad_sch" (at 25.4 50.1146 0)
-      (effects (font (size 1.27 1.27)) (justify left top))
-    )
-    (instances
-      (project "overall scematic"
-        (path "/9230863d-68c5-4e85-a5d4-0f54ecfbae5b" (page "2"))
-      )
     )
   )

Commit message: updated schematic
Parts:
- added BT1: Battery_Cell, symbol Device:Battery_Cell
Connections:
- new net Battery+: BT1.1 (+)
- new net Battery-: BT1.2 (-)
Changed lines of the file:
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@@
     (rev "version1")
+  )
+  (hierarchical_label "3v3" (shape output) (at 241.3 121.92 270) (fields_autoplaced)
+    (effects (font (size 1.27 1.27)) (justify right))
+  )
+  (hierarchical_label "Battery-" (shape bidirectional) (at 191.77 133.35 270) (fields_autoplaced)
+    (effects (font (size 1.27 1.27)) (justify right))
+  )
+  (hierarchical_label "Battery+" (shape bidirectional) (at 191.77 125.73 90) (fields_autoplaced)
+    (effects (font (size 1.27 1.27)) (justify left))
+  )
+  (symbol (lib_id "Device:Battery_Cell") (at 191.77 130.81 0) (unit 1)
+    (in_bom yes) (on_board yes) (dnp no) (fields_autoplaced)
+    (property "Reference" "BT1" (at 195.58 128.143 0)
+      (effects (font (size 1.27 1.27)) (justify left))
+    )
+    (property "Value" "Battery_Cell" (at 195.58 130.683 0)
+      (effects (font (size 1.27 1.27)) (justify left))
+    )
+    (property "Footprint" "" (at 191.77 129.286 90)
+      (effects (font (size 1.27 1.27)) hide)
+    )
+    (property "Datasheet" "~" (at 191.77 129.286 90)
+      (effects (font (size 1.27 1.27)) hide)
+    )
+    (pin "1")
+    (pin "2")
+    (instances
+      (project "overall scematic"
+        (path "/9230863d-68c5-4e85-a5d4-0f54ecfbae5b"
+          (reference "BT1") (unit 1)
+        )
+      )
+    )
+  )
+  (symbol (lib_id "power:+3V3") (at 241.3 121.92 0) (unit 1)
+    (in_bom yes) (on_board yes) (dnp no) (fields_autoplaced)
+    (property "Reference" "#PWR013" (at 241.3 125.73 0)
+      (effects (font (size 1.27 1.27)) hide)
+    )
+    (property "Value" "+3V3" (at 241.3 118.11 0)
+      (effects (font (size 1.27 1.27)))
+    )
+    (property "Footprint" "" (at 241.3 121.92 0)
+      (effects (font (size 1.27 1.27)) hide)
+    )
+    (property "Datasheet" "" (at 241.3 121.92 0)
+      (effects (font (size 1.27 1.27)) hide)
+    )
+    (pin "1")
+    (instances
+      (project "overall scematic"
+        (path "/9230863d-68c5-4e85-a5d4-0f54ecfbae5b"
+          (reference "#PWR013") (unit 1)
+        )
+      )
+    )
+  )
+  (symbol (lib_id "power:PWR_FLAG") (at 231.14 121.92 180) (unit 1)
+    (in_bom yes) (on_board yes) (dnp no) (fields_autoplaced)
+    (property "Reference" "#FLG02" (at 231.14 123.825 0)
+      (effects (font (size 1.27 1.27)) hide)
+    )
+    (property "Value" "PWR_FLAG" (at 231.14 127 0)
+      (effects (font (size 1.27 1.27)))
+    )
+    (property "Footprint" "" (at 231.14 121.92 0)
+      (effects (font (size 1.27 1.27)) hide)
+    )
+    (property "Datasheet" "~" (at 231.14 121.92 0)
+      (effects (font (size 1.27 1.27)) hide)
+    )
+    (pin "1")
+    (instances
+      (project "overall scematic"
+        (path "/9230863d-68c5-4e85-a5d4-0f54ecfbae5b"
+          (reference "#FLG02") (unit 1)
+        )
+      )
+    )
+  )
+  (symbol (lib_id "power:+5V") (at 231.14 121.92 0) (unit 1)
+    (in_bom yes) (on_board yes) (dnp no) (fields_autoplaced)
+    (property "Reference" "#PWR012" (at 231.14 125.73 0)
+      (effects (font (size 1.27 1.27)) hide)
+    )
+    (property "Value" "+5V" (at 231.14 118.11 0)
+      (effects (font (size 1.27 1.27)))
+    )
+    (property "Footprint" "" (at 231.14 121.92 0)
+      (effects (font (size 1.27 1.27)) hide)
+    )
+    (property "Datasheet" "" (at 231.14 121.92 0)
+      (effects (font (size 1.27 1.27)) hide)
+    )
+    (pin "1")
+    (instances
+      (project "overall scematic"
+        (path "/9230863d-68c5-4e85-a5d4-0f54ecfbae5b"
+          (reference "#PWR012") (unit 1)
+        )
+      )
+    )
+  )
+  (symbol (lib_id "power:VDD") (at 218.44 121.92 0) (unit 1)
+    (in_bom yes) (on_board yes) (dnp no) (fields_autoplaced)
+    (property "Reference" "#PWR011" (at 218.44 125.73 0)
+      (effects (font (size 1.27 1.27)) hide)
+    )
+    (property "Value" "VDD" (at 218.44 118.11 0)
+      (effects (font (size 1.27 1.27)))
+    )
+    (property "Footprint" "" (at 218.44 121.92 0)
+      (effects (font (size 1.27 1.27)) hide)
+    )
+    (property "Datasheet" "" (at 218.44 121.92 0)
+      (effects (font (size 1.27 1.27)) hide)
+    )
+    (pin "1")
+    (instances
+      (project "overall scematic"
+        (path "/9230863d-68c5-4e85-a5d4-0f54ecfbae5b"
+          (reference "#PWR011") (unit 1)
+        )
+      )
+    )
+  )
+  (symbol (lib_id "power:PWR_FLAG") (at 218.44 121.92 180) (unit 1)
+    (in_bom yes) (on_board yes) (dnp no) (fields_autoplaced)
+    (property "Reference" "#FLG01" (at 218.44 123.825 0)
+      (effects (font (size 1.27 1.27)) hide)
+    )
+    (property "Value" "PWR_FLAG" (at 218.44 127 0)
+      (effects (font (size 1.27 1.27)))
+    )
+    (property "Footprint" "" (at 218.44 121.92 0)
+      (effects (font (size 1.27 1.27)) hide)
+    )
+    (property "Datasheet" "~" (at 218.44 121.92 0)
+      (effects (font (size 1.27 1.27)) hide)
+    )
+    (pin "1")
+    (instances
+      (project "overall scematic"
+        (path "/9230863d-68c5-4e85-a5d4-0f54ecfbae5b"
+          (reference "#FLG01") (unit 1)
+        )
+      )
+    )
   )
   (sheet (at 25.4 60.96) (size 54.61 17.78) (fields_autoplaced)
