File: Overall schematic/overall scematic/overall scematic.kicad_sch (KiCad schematic)
At the start: 1 part

Commit message: Add files via upload
Other:
- sheet digital temparature sensor renamed digital sensor(Humidity and Temperature
- removed sheet Humidity sensor
- sheet digital sensor(Humidity and Temperature ports: added none; removed SCL, SDA, Supply Voltage
Changed lines of the file:
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@@
-    )
-  )
-  (sheet (at 25.4 60.96) (size 54.61 17.78) (fields_autoplaced)
-    (stroke (width 0.1524) (type solid))
-    (fill (color 0 0 0 0.0000))
-    (property "Sheetname" "Humidity sensor" (at 25.4 60.2484 0)
-      (effects (font (size 1.27 1.27)) (justify left bottom))
-    )
-    (property "Sheetfile" "digital_sensor.kicad_sch" (at 25.4 79.3246 0)
-      (effects (font (size 1.27 1.27)) (justify left top))
-    )
-    (instances
-      (project "overall scematic"
-        (path "/9230863d-68c5-4e85-a5d4-0f54ecfbae5b" (page "3"))
-      )
     )
   )
@@
     )
   )
-  (sheet (at 26.67 114.3) (size 53.34 13.97) (fields_autoplaced)
+  (sheet (at 26.67 113.03) (size 53.34 13.97) (fields_autoplaced)
     (stroke (width 0.1524) (type solid))
     (fill (color 0 0 0 0.0000))
-    (property "Sheetname" "digital temparature sensor" (at 26.67 113.5884 0)
+    (property "Sheetname" "digital sensor(Humidity and Temperature" (at 26.67 112.3184 0)
       (effects (font (size 1.27 1.27)) (justify left bottom))
     )
-    (property "Sheetfile" "digi temp.kicad_sch" (at 26.67 128.8546 0)
+    (property "Sheetfile" "digi temp.kicad_sch" (at 26.67 127.5846 0)
       (effects (font (size 1.27 1.27)) (justify left top))
     )
-    (pin "Supply Voltage" input (at 26.67 118.11 180)
-      (effects (font (size 1.27 1.27)) (justify left))
-    )
-    (pin "SCL" input (at 80.01 121.92 0)
-      (effects (font (size 1.27 1.27)) (justify right))
-    )
-    (pin "SDA" input (at 80.01 119.38 0)
-      (effects (font (size 1.27 1.27)) (justify right))
-    )
     (instances

Commit message: fully annotated
Other:
- sheet Micro controller pin outs ports: added Analogue_out, SCL, SDA; removed none
- sheet Power module ports: added Battery+, Battery-, Supply_Voltage; removed none
- sheet analogue temparature sensor ports: added Analogue_out, Supply Voltage; removed none
- sheet digital sensor(Humidity and Temperature ports: added SCL, SDA, Supply_Voltage; removed none

Commit message: updated everything
Parts:
- BT1: footprint (none) -> Battery:BatteryHolder_Keystone_2466_1xAAA
Other:
- sheet Micro controller pin outs ports: added Supply_Voltage; removed none
- sheet analogue temparature sensor ports: added Supply_Voltage; removed Supply Voltage
Changed lines of the file:
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@@
     (rev "version1")
   )
-  (junction (at 83.82 115.57) (diameter 0) (color 0 0 0 0)
-  )
-  (junction (at 85.09 97.79) (diameter 0) (color 0 0 0 0)
-  )
-  (junction (at 196.85 39.37) (diameter 0) (color 0 0 0 0)
-  )
   (wire (pts (xy 191.77 115.57) (xy 191.77 125.73))
     (stroke (width 0) (type default))
@@
     (stroke (width 0) (type default))
   )
-  (wire (pts (xy 193.04 39.37) (xy 196.85 39.37))
-    (stroke (width 0) (type default))
-  )
-  (wire (pts (xy 80.01 97.79) (xy 85.09 97.79))
+  (wire (pts (xy 193.04 39.37) (xy 209.55 39.37))
     (stroke (width 0) (type default))
   )
@@
     (stroke (width 0) (type default))
   )
-  (wire (pts (xy 80.01 115.57) (xy 83.82 115.57))
+  (wire (pts (xy 80.01 97.79) (xy 93.98 97.79))
+    (stroke (width 0) (type default))
+  )
+  (wire (pts (xy 80.01 115.57) (xy 99.06 115.57))
     (stroke (width 0) (type default))
   )
@@
     (stroke (width 0) (type default))
   )
+  (wire (pts (xy 109.22 78.74) (xy 127 78.74))
+    (stroke (width 0) (type default))
+  )
   (wire (pts (xy 80.01 120.65) (xy 86.36 120.65))
     (stroke (width 0) (type default))
   )
-  (wire (pts (xy 196.85 39.37) (xy 201.93 39.37))
-    (stroke (width 0) (type default))
-  )
   (wire (pts (xy 191.77 140.97) (xy 191.77 133.35))
     (stroke (width 0) (type default))
@@
     (stroke (width 0) (type default))
   )
-  (wire (pts (xy 83.82 115.57) (xy 92.71 115.57))
-    (stroke (width 0) (type default))
-  )
   (wire (pts (xy 193.04 44.45) (xy 201.93 44.45))
     (stroke (width 0) (type default))
   )
-  (wire (pts (xy 85.09 97.79) (xy 93.98 97.79))
-    (stroke (width 0) (type default))
+  (label "Supply_Voltage" (at 93.98 97.79 180) (fields_autoplaced)
+    (effects (font (size 1.27 1.27)) (justify right bottom))
   )
   (label "Battery+" (at 191.77 124.46 90) (fields_autoplaced)
@@
     (effects (font (size 1.27 1.27)) (justify right bottom))
   )
-  (label "Battery-" (at 201.93 41.91 0) (fields_autoplaced)
-    (effects (font (size 1.27 1.27)) (justify left bottom))
+  (label "Supply_Voltage" (at 99.06 115.57 180) (fields_autoplaced)
+    (effects (font (size 1.27 1.27)) (justify right bottom))
+  )
+  (label "Supply_Voltage" (at 109.22 78.74 0) (fields_autoplaced)
+    (effects (font (size 1.27 1.27)) (justify left bottom))
+  )
+  (label "Supply_Voltage" (at 209.55 39.37 180) (fields_autoplaced)
+    (effects (font (size 1.27 1.27)) (justify right bottom))
+  )
+  (label "Battery-" (at 201.93 41.91 180) (fields_autoplaced)
+    (effects (font (size 1.27 1.27)) (justify right bottom))
   )
   (label "SCL" (at 121.92 86.36 0) (fields_autoplaced)
     (effects (font (size 1.27 1.27)) (justify left bottom))
   )
-  (label "Battery+" (at 201.93 44.45 0) (fields_autoplaced)
-    (effects (font (size 1.27 1.27)) (justify left bottom))
+  (label "Battery+" (at 201.93 44.45 180) (fields_autoplaced)
+    (effects (font (size 1.27 1.27)) (justify right bottom))
   )
   (label "SCL" (at 86.36 120.65 180) (fields_autoplaced)
@@
       (effects (font (size 1.27 1.27)) (justify left))
     )
-    (property "Footprint" "" (at 191.77 129.286 90)
+    (property "Footprint" "Battery:BatteryHolder_Keystone_2466_1xAAA" (at 191.77 129.286 90)
       (effects (font (size 1.27 1.27)) hide)
     )
@@
     )
   )
-  (symbol (lib_id "power:PWR_FLAG") (at 201.93 39.37 270) (unit 1)
-    (in_bom yes) (on_board yes) (dnp no) (fields_autoplaced)
-    (property "Reference" "#FLG02" (at 203.835 39.37 0)
-      (effects (font (size 1.27 1.27)) hide)
-    )
-    (property "Value" "PWR_FLAG" (at 205.74 40.005 90)
-      (effects (font (size 1.27 1.27)) (justify left))
-    )
-    (property "Footprint" "" (at 201.93 39.37 0)
-      (effects (font (size 1.27 1.27)) hide)
-    )
-    (property "Datasheet" "~" (at 201.93 39.37 0)
-      (effects (font (size 1.27 1.27)) hide)
-    )
-    (pin "1")
-    (instances
-      (project "overall scematic"
-        (path "/9230863d-68c5-4e85-a5d4-0f54ecfbae5b"
-          (reference "#FLG02") (unit 1)
-        )
-      )
-    )
-  )
-  (symbol (lib_id "power:PWR_FLAG") (at 85.09 97.79 0) (unit 1)
-    (in_bom yes) (on_board yes) (dnp no) (fields_autoplaced)
-    (property "Reference" "#FLG06" (at 85.09 95.885 0)
-      (effects (font (size 1.27 1.27)) hide)
-    )
-    (property "Value" "PWR_FLAG" (at 85.09 93.98 0)
-      (effects (font (size 1.27 1.27)))
-    )
-    (property "Footprint" "" (at 85.09 97.79 0)
-      (effects (font (size 1.27 1.27)) hide)
-    )
-    (property "Datasheet" "~" (at 85.09 97.79 0)
-      (effects (font (size 1.27 1.27)) hide)
-    )
-    (pin "1")
-    (instances
-      (project "overall scematic"
-        (path "/9230863d-68c5-4e85-a5d4-0f54ecfbae5b"
-          (reference "#FLG06") (unit 1)
-        )
-      )
-    )
-  )
-  (symbol (lib_id "power:VDD") (at 218.44 30.48 0) (unit 1)
-    (in_bom yes) (on_board yes) (dnp no) (fields_autoplaced)
-    (property "Reference" "#PWR011" (at 218.44 34.29 0)
-      (effects (font (size 1.27 1.27)) hide)
-    )
-    (property "Value" "VDD" (at 218.44 26.67 0)
-      (effects (font (size 1.27 1.27)))
-    )
-    (property "Footprint" "" (at 218.44 30.48 0)
-      (effects (font (size 1.27 1.27)) hide)
-    )
-    (property "Datasheet" "" (at 218.44 30.48 0)
-      (effects (font (size 1.27 1.27)) hide)
-    )
-    (pin "1")
-    (instances
-      (project "overall scematic"
-        (path "/9230863d-68c5-4e85-a5d4-0f54ecfbae5b"
-          (reference "#PWR011") (unit 1)
-        )
-      )
-    )
-  )
-  (symbol (lib_id "power:VDD") (at 93.98 97.79 0) (unit 1)
-    (in_bom yes) (on_board yes) (dnp no) (fields_autoplaced)
-    (property "Reference" "#PWR07" (at 93.98 101.6 0)
-      (effects (font (size 1.27 1.27)) hide)
-    )
-    (property "Value" "VDD" (at 93.98 93.98 0)
-      (effects (font (size 1.27 1.27)))
-    )
-    (property "Footprint" "" (at 93.98 97.79 0)
-      (effects (font (size 1.27 1.27)) hide)
-    )
-    (property "Datasheet" "" (at 93.98 97.79 0)
-      (effects (font (size 1.27 1.27)) hide)
-    )
-    (pin "1")
-    (instances
-      (project "overall scematic"
-        (path "/9230863d-68c5-4e85-a5d4-0f54ecfbae5b"
-          (reference "#PWR07") (unit 1)
-        )
-      )
-    )
-  )
-  (symbol (lib_id "power:PWR_FLAG") (at 218.44 30.48 180) (unit 1)
-    (in_bom yes) (on_board yes) (dnp no) (fields_autoplaced)
-    (property "Reference" "#FLG01" (at 218.44 32.385 0)
-      (effects (font (size 1.27 1.27)) hide)
-    )
-    (property "Value" "PWR_FLAG" (at 218.44 35.56 0)
-      (effects (font (size 1.27 1.27)))
-    )
-    (property "Footprint" "" (at 218.44 30.48 0)
-      (effects (font (size 1.27 1.27)) hide)
-    )
-    (property "Datasheet" "~" (at 218.44 30.48 0)
-      (effects (font (size 1.27 1.27)) hide)
-    )
-    (pin "1")
-    (instances
-      (project "overall scematic"
-        (path "/9230863d-68c5-4e85-a5d4-0f54ecfbae5b"
-          (reference "#FLG01") (unit 1)
-        )
-      )
-    )
-  )
-  (symbol (lib_id "power:PWR_FLAG") (at 83.82 115.57 0) (unit 1)
-    (in_bom yes) (on_board yes) (dnp no) (fields_autoplaced)
-    (property "Reference" "#FLG07" (at 83.82 113.665 0)
-      (effects (font (size 1.27 1.27)) hide)
-    )
-    (property "Value" "PWR_FLAG" (at 83.82 111.76 0)
-      (effects (font (size 1.27 1.27)))
-    )
-    (property "Footprint" "" (at 83.82 115.57 0)
-      (effects (font (size 1.27 1.27)) hide)
-    )
-    (property "Datasheet" "~" (at 83.82 115.57 0)
-      (effects (font (size 1.27 1.27)) hide)
-    )
-    (pin "1")
-    (instances
-      (project "overall scematic"
-        (path "/9230863d-68c5-4e85-a5d4-0f54ecfbae5b"
-          (reference "#FLG07") (unit 1)
-        )
-      )
-    )
-  )
-  (symbol (lib_id "power:VDD") (at 196.85 39.37 0) (unit 1)
-    (in_bom yes) (on_board yes) (dnp no) (fields_autoplaced)
-    (property "Reference" "#PWR06" (at 196.85 43.18 0)
-      (effects (font (size 1.27 1.27)) hide)
-    )
-    (property "Value" "VDD" (at 196.85 35.56 0)
-      (effects (font (size 1.27 1.27)))
-    )
-    (property "Footprint" "" (at 196.85 39.37 0)
-      (effects (font (size 1.27 1.27)) hide)
-    )
-    (property "Datasheet" "" (at 196.85 39.37 0)
-      (effects (font (size 1.27 1.27)) hide)
-    )
-    (pin "1")
-    (instances
-      (project "overall scematic"
-        (path "/9230863d-68c5-4e85-a5d4-0f54ecfbae5b"
-          (reference "#PWR06") (unit 1)
-        )
-      )
-    )
-  )
-  (symbol (lib_id "power:VDD") (at 92.71 115.57 0) (unit 1)
-    (in_bom yes) (on_board yes) (dnp no) (fields_autoplaced)
-    (property "Reference" "#PWR08" (at 92.71 119.38 0)
-      (effects (font (size 1.27 1.27)) hide)
-    )
-    (property "Value" "VDD" (at 92.71 111.76 0)
-      (effects (font (size 1.27 1.27)))
-    )
-    (property "Footprint" "" (at 92.71 115.57 0)
-      (effects (font (size 1.27 1.27)) hide)
-    )
-    (property "Datasheet" "" (at 92.71 115.57 0)
-      (effects (font (size 1.27 1.27)) hide)
-    )
-    (pin "1")
-    (instances
-      (project "overall scematic"
-        (path "/9230863d-68c5-4e85-a5d4-0f54ecfbae5b"
-          (reference "#PWR08") (unit 1)
-        )
-      )
-    )
-  )
   (sheet (at 125.73 24.13) (size 67.31 25.4) (fields_autoplaced)
     (stroke (width 0.1524) (type solid))
@@
       (effects (font (size 1.27 1.27)) (justify left))
     )
+    (pin "Supply_Voltage" input (at 127 78.74 180)
+      (effects (font (size 1.27 1.27)) (justify left))
+    )
     (instances
       (project "overall scematic"
@@
       (effects (font (size 1.27 1.27)) (justify right))
     )
-    (pin "Supply Voltage" input (at 80.01 97.79 0)
-      (effects (font (size 1.27 1.27)) (justify right))
-    )
+    (pin "Supply_Voltage" input (at 80.01 97.79 0)
+      (effects (font (size 1.27 1.27)) (justify right))
+    )

Commit message: BOM
Other:
- company: (none) -> University of capetown
- title: overall schematic -> 3088_group22_design
Changed lines of the file:
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@@
   (paper "A4")
   (title_block
-    (title "overall schematic")
-    (date "2023-03-10")
-    (rev "version1")
+    (title "3088_group22_design")
+    (date "2023-03-20")
+    (rev "3")
+    (company "University of capetown")
   )
   (wire (pts (xy 191.77 115.57) (xy 191.77 125.73))

Commit message: hail mary
Parts:
- BT1: footprint Battery:BatteryHolder_Keystone_2466_1xAAA -> BAT60JFILM:18650_Holder_SMD
Changed lines of the file:
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@@
       (effects (font (size 1.27 1.27)) (justify left))
     )
-    (property "Footprint" "Battery:BatteryHolder_Keystone_2466_1xAAA" (at 191.77 129.286 90)
+    (property "Footprint" "BAT60JFILM:18650_Holder_SMD" (at 191.77 129.286 90)
       (effects (font (size 1.27 1.27)) hide)
     )
