File: Overall schematic/overall scematic/analogue_temparature.kicad_sch (KiCad schematic)
At the start: 0 parts

Commit message: Add files via upload
Parts:
- added U?: MCP9701AT-E_TT, digikey-footprints:SOT-23-3, symbol dk_Temperature-Sensors-Analog-and-Digital-Output:MCP9701AT-E_TT
Connections:
- new net GND: U?.3 (GND)
- new net PAx: U?.2 (VOUT)
- new net Vreg_Out: U?.1 (VDD)
Changed lines of the file:
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@@
 (kicad_sch (version 20230121) (generator eeschema)
   (paper "A4")
+  (wire (pts (xy 115.57 96.52) (xy 120.65 96.52))
+    (stroke (width 0) (type default))
+  )
+  (wire (pts (xy 105.41 104.14) (xy 105.41 106.68))
+    (stroke (width 0) (type default))
+  )
+  (global_label "PAx" (shape output) (at 120.65 96.52 0) (fields_autoplaced)
+    (effects (font (size 1.27 1.27)) (justify left))
+    (property "Intersheetrefs" "${INTERSHEET_REFS}" (at 126.9425 96.52 0)
+      (effects (font (size 1.27 1.27)) (justify left) hide)
+    )
+  )
+  (global_label "Vreg_Out" (shape input) (at 105.41 88.9 90) (fields_autoplaced)
+    (effects (font (size 1.27 1.27)) (justify left))
+    (property "Intersheetrefs" "${INTERSHEET_REFS}" (at 105.41 77.709 90)
+      (effects (font (size 1.27 1.27)) (justify left) hide)
+    )
+  )
+  (symbol (lib_id "dk_Temperature-Sensors-Analog-and-Digital-Output:MCP9701AT-E_TT") (at 105.41 96.52 0) (unit 1)
+    (in_bom yes) (on_board yes) (dnp no) (fields_autoplaced)
+    (property "Reference" "U?" (at 101.6 95.885 0)
+      (effects (font (size 1.524 1.524)) (justify right))
+    )
+    (property "Value" "MCP9701AT-E_TT" (at 101.6 98.425 0)
+      (effects (font (size 1.524 1.524)) (justify right))
+    )
+    (property "Footprint" "digikey-footprints:SOT-23-3" (at 110.49 91.44 0)
+      (effects (font (size 1.524 1.524)) (justify left) hide)
+    )
+    (property "Datasheet" "http://www.microchip.com/mymicrochip/filehandler.aspx?ddocname=en022859" (at 110.49 88.9 0)
+      (effects (font (size 1.524 1.524)) (justify left) hide)
+    )
+    (property "Digi-Key_PN" "MCP9701AT-E/TTCT-ND" (at 110.49 86.36 0)
+      (effects (font (size 1.524 1.524)) (justify left) hide)
+    )
+    (property "MPN" "MCP9701AT-E/TT" (at 110.49 83.82 0)
+      (effects (font (size 1.524 1.524)) (justify left) hide)
+    )
+    (property "Category" "Sensors, Transducers" (at 110.49 81.28 0)
+      (effects (font (size 1.524 1.524)) (justify left) hide)
+    )
+    (property "Family" "Temperature Sensors - Analog and Digital Output" (at 110.49 78.74 0)
+      (effects (font (size 1.524 1.524)) (justify left) hide)
+    )
+    (property "DK_Datasheet_Link" "http://www.microchip.com/mymicrochip/filehandler.aspx?ddocname=en022859" (at 110.49 76.2 0)
+      (effects (font (size 1.524 1.524)) (justify left) hide)
+    )
+    (property "DK_Detail_Page" "/product-detail/en/microchip-technology/MCP9701AT-E-TT/MCP9701AT-E-TTCT-ND/1987449" (at 110.49 73.66 0)
+      (effects (font (size 1.524 1.524)) (justify left) hide)
+    )
+    (property "Description" "SENSOR ANALOG -10C-125C SOT23-3" (at 110.49 71.12 0)
+      (effects (font (size 1.524 1.524)) (justify left) hide)
+    )
+    (property "Manufacturer" "Microchip Technology" (at 110.49 68.58 0)
+      (effects (font (size 1.524 1.524)) (justify left) hide)
+    )
+    (property "Status" "Active" (at 110.49 66.04 0)
+      (effects (font (size 1.524 1.524)) (justify left) hide)
+    )
+    (pin "1")
+    (pin "2")
+    (pin "3")
+    (instances
+      (project "overall scematic"
+        (path "/9230863d-68c5-4e85-a5d4-0f54ecfbae5b/c494e013-0c38-49c8-84da-4f33138ae19d"
+          (reference "U?") (unit 1)
+        )
+      )
+      (project "analogue_temparature"
+        (path "/fd616d34-a44b-4530-b77b-84bccfccd64d"
+          (reference "U?") (unit 1)
+        )
+      )
+    )
+  )
+  (symbol (lib_id "power:GND") (at 105.41 106.68 0) (unit 1)
+    (in_bom yes) (on_board yes) (dnp no) (fields_autoplaced)
+    (property "Reference" "#PWR?" (at 105.41 113.03 0)
+      (effects (font (size 1.27 1.27)) hide)
+    )
+    (property "Value" "GND" (at 105.41 111.76 0)
+      (effects (font (size 1.27 1.27)))
+    )
+    (property "Footprint" "" (at 105.41 106.68 0)
+      (effects (font (size 1.27 1.27)) hide)
+    )
+    (property "Datasheet" "" (at 105.41 106.68 0)
+      (effects (font (size 1.27 1.27)) hide)
+    )
+    (pin "1")
+    (instances
+      (project "overall scematic"
+        (path "/9230863d-68c5-4e85-a5d4-0f54ecfbae5b/c494e013-0c38-49c8-84da-4f33138ae19d"
+          (reference "#PWR?") (unit 1)
+        )
+      )
+      (project "analogue_temparature"
+        (path "/fd616d34-a44b-4530-b77b-84bccfccd64d"
+          (reference "#PWR?") (unit 1)
+        )
+      )
+    )
+  )
+  (sheet_instances
+    (path "/" (page "1"))
+  )
 )

Commit message: updated schematic
Changed lines of the file:
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@@
     (stroke (width 0) (type default))
   )
-  (global_label "PAx" (shape output) (at 120.65 96.52 0) (fields_autoplaced)
+  (hierarchical_label "Vreg_Out" (shape input) (at 105.41 88.9 90) (fields_autoplaced)
     (effects (font (size 1.27 1.27)) (justify left))
-    (property "Intersheetrefs" "${INTERSHEET_REFS}" (at 126.9425 96.52 0)
-      (effects (font (size 1.27 1.27)) (justify left) hide)
-    )
   )
-  (global_label "Vreg_Out" (shape input) (at 105.41 88.9 90) (fields_autoplaced)
+  (hierarchical_label "PAx" (shape input) (at 120.65 96.52 0) (fields_autoplaced)
     (effects (font (size 1.27 1.27)) (justify left))
-    (property "Intersheetrefs" "${INTERSHEET_REFS}" (at 105.41 77.709 90)
-      (effects (font (size 1.27 1.27)) (justify left) hide)
-    )
   )
   (symbol (lib_id "dk_Temperature-Sensors-Analog-and-Digital-Output:MCP9701AT-E_TT") (at 105.41 96.52 0) (unit 1)

Commit message: Add files via upload
Parts:
- gave numbers to parts that had none: 1
Connections:
- net Vreg_Out renamed Supply Voltage
Changed lines of the file:
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@@
 (kicad_sch (version 20230121) (generator eeschema)
   (paper "A4")
+  (wire (pts (xy 105.41 82.55) (xy 105.41 88.9))
+    (stroke (width 0) (type default))
+  )
   (wire (pts (xy 115.57 96.52) (xy 120.65 96.52))
     (stroke (width 0) (type default))
@@
     (stroke (width 0) (type default))
   )
-  (hierarchical_label "Vreg_Out" (shape input) (at 105.41 88.9 90) (fields_autoplaced)
+  (global_label "PAx" (shape output) (at 120.65 96.52 0) (fields_autoplaced)
     (effects (font (size 1.27 1.27)) (justify left))
+    (property "Intersheetrefs" "${INTERSHEET_REFS}" (at 126.9425 96.52 0)
+      (effects (font (size 1.27 1.27)) (justify left) hide)
+    )
   )
-  (hierarchical_label "PAx" (shape input) (at 120.65 96.52 0) (fields_autoplaced)
+  (global_label "Supply Voltage" (shape input) (at 105.41 82.55 90) (fields_autoplaced)
     (effects (font (size 1.27 1.27)) (justify left))
+    (property "Intersheetrefs" "${INTERSHEET_REFS}" (at 105.41 65.5778 90)
+      (effects (font (size 1.27 1.27)) (justify left) hide)
+    )
   )
   (symbol (lib_id "dk_Temperature-Sensors-Analog-and-Digital-Output:MCP9701AT-E_TT") (at 105.41 96.52 0) (unit 1)
-    (in_bom yes) (on_board yes) (dnp no) (fields_autoplaced)
-    (property "Reference" "U?" (at 101.6 95.885 0)
+    (in_bom yes) (on_board yes) (dnp no)
+    (property "Reference" "U5" (at 101.6 95.885 0)
       (effects (font (size 1.524 1.524)) (justify right))
     )
@@
       (project "overall scematic"
         (path "/9230863d-68c5-4e85-a5d4-0f54ecfbae5b/c494e013-0c38-49c8-84da-4f33138ae19d"
-          (reference "U?") (unit 1)
+          (reference "U5") (unit 1)
         )
       )

Commit message: fully annotated
Connections:
- net PAx renamed Analogue_out
Changed lines of the file:
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@@
     (stroke (width 0) (type default))
   )
-  (global_label "PAx" (shape output) (at 120.65 96.52 0) (fields_autoplaced)
+  (hierarchical_label "Supply Voltage" (shape input) (at 105.41 82.55 90) (fields_autoplaced)
     (effects (font (size 1.27 1.27)) (justify left))
-    (property "Intersheetrefs" "${INTERSHEET_REFS}" (at 126.9425 96.52 0)
-      (effects (font (size 1.27 1.27)) (justify left) hide)
-    )
   )
-  (global_label "Supply Voltage" (shape input) (at 105.41 82.55 90) (fields_autoplaced)
+  (hierarchical_label "Analogue_out" (shape output) (at 120.65 96.52 0) (fields_autoplaced)
     (effects (font (size 1.27 1.27)) (justify left))
-    (property "Intersheetrefs" "${INTERSHEET_REFS}" (at 105.41 65.5778 90)
-      (effects (font (size 1.27 1.27)) (justify left) hide)
-    )
   )
   (symbol (lib_id "dk_Temperature-Sensors-Analog-and-Digital-Output:MCP9701AT-E_TT") (at 105.41 96.52 0) (unit 1)
@@
   (symbol (lib_id "power:GND") (at 105.41 106.68 0) (unit 1)
     (in_bom yes) (on_board yes) (dnp no) (fields_autoplaced)
-    (property "Reference" "#PWR?" (at 105.41 113.03 0)
+    (property "Reference" "#PWR09" (at 105.41 113.03 0)
       (effects (font (size 1.27 1.27)) hide)
     )
@@
       (project "overall scematic"
         (path "/9230863d-68c5-4e85-a5d4-0f54ecfbae5b/c494e013-0c38-49c8-84da-4f33138ae19d"
-          (reference "#PWR?") (unit 1)
+          (reference "#PWR09") (unit 1)
         )
       )

Commit message: updated everything
Parts:
- U5: footprint digikey-footprints:SOT-23-3 -> MCP9701AT-E_TT:SOT-23-3
Connections:
- net Supply Voltage renamed Supply_Voltage
Changed lines of the file:
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@@
     (stroke (width 0) (type default))
   )
-  (hierarchical_label "Supply Voltage" (shape input) (at 105.41 82.55 90) (fields_autoplaced)
+  (hierarchical_label "Supply_Voltage" (shape input) (at 105.41 82.55 90) (fields_autoplaced)
     (effects (font (size 1.27 1.27)) (justify left))
   )
@@
       (effects (font (size 1.524 1.524)) (justify right))
     )
-    (property "Footprint" "digikey-footprints:SOT-23-3" (at 110.49 91.44 0)
+    (property "Footprint" "MCP9701AT-E_TT:SOT-23-3" (at 110.49 91.44 0)
       (effects (font (size 1.524 1.524)) (justify left) hide)
     )

Commit message: BOM
Other:
- company: (none) -> University of capetown
- title: (none) -> 3088_group22_design
Changed lines of the file:
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@@
 (kicad_sch (version 20230121) (generator eeschema)
   (paper "A4")
+  (title_block
+    (title "3088_group22_design")
+    (date "2023-03-20")
+    (rev "3")
+    (company "University of capetown")
+  )
   (wire (pts (xy 105.41 82.55) (xy 105.41 88.9))
     (stroke (width 0) (type default))

Commit message: The final Gerber
Changed lines of the file:
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@@
     (company "University of capetown")
+  )
+  (wire (pts (xy 119.38 91.44) (xy 128.27 91.44))
+    (stroke (width 0) (type default))
+  )
+  (wire (pts (xy 128.27 91.44) (xy 128.27 88.9))
+    (stroke (width 0) (type default))
+  )
+  (wire (pts (xy 119.38 82.55) (xy 119.38 91.44))
+    (stroke (width 0) (type default))
   )
   (wire (pts (xy 105.41 82.55) (xy 105.41 88.9))
@@
     (stroke (width 0) (type default))
   )
+  (hierarchical_label "Supply_Voltage" (shape input) (at 128.27 88.9 90) (fields_autoplaced)
+    (effects (font (size 1.27 1.27)) (justify left))
+  )
   (hierarchical_label "Supply_Voltage" (shape input) (at 105.41 82.55 90) (fields_autoplaced)
     (effects (font (size 1.27 1.27)) (justify left))
@@
   (hierarchical_label "Analogue_out" (shape output) (at 120.65 96.52 0) (fields_autoplaced)
     (effects (font (size 1.27 1.27)) (justify left))
+  )
+  (symbol (lib_id "power:PWR_FLAG") (at 119.38 82.55 0) (unit 1)
+    (in_bom yes) (on_board yes) (dnp no) (fields_autoplaced)
+    (property "Reference" "#FLG0101" (at 119.38 80.645 0)
+      (effects (font (size 1.27 1.27)) hide)
+    )
+    (property "Value" "PWR_FLAG" (at 119.38 78.74 0)
+      (effects (font (size 1.27 1.27)))
+    )
+    (property "Footprint" "" (at 119.38 82.55 0)
+      (effects (font (size 1.27 1.27)) hide)
+    )
+    (property "Datasheet" "~" (at 119.38 82.55 0)
+      (effects (font (size 1.27 1.27)) hide)
+    )
+    (pin "1")
+    (instances
+      (project "overall scematic"
+        (path "/9230863d-68c5-4e85-a5d4-0f54ecfbae5b/c494e013-0c38-49c8-84da-4f33138ae19d"
+          (reference "#FLG0101") (unit 1)
+        )
+      )
+    )
   )
   (symbol (lib_id "dk_Temperature-Sensors-Analog-and-Digital-Output:MCP9701AT-E_TT") (at 105.41 96.52 0) (unit 1)
@@
   (symbol (lib_id "power:GND") (at 105.41 106.68 0) (unit 1)
     (in_bom yes) (on_board yes) (dnp no) (fields_autoplaced)
-    (property "Reference" "#PWR09" (at 105.41 113.03 0)
+    (property "Reference" "#PWR0101" (at 105.41 113.03 0)
       (effects (font (size 1.27 1.27)) hide)
     )
@@
       (project "overall scematic"
         (path "/9230863d-68c5-4e85-a5d4-0f54ecfbae5b/c494e013-0c38-49c8-84da-4f33138ae19d"
-          (reference "#PWR09") (unit 1)
+          (reference "#PWR0101") (unit 1)
         )
       )
