File: Overall schematic/overall scematic/analogue_temparature.kicad_sch (KiCad schematic)
At the start: 1 part, among them U5 MCP9701AT-E_TT

Commit message: hail mary
Parts:
- U5: footprint MCP9701AT-E_TT:SOT-23-3 -> BAT60JFILM:SOT-23-3
Changed lines of the file:
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@@
       (effects (font (size 1.524 1.524)) (justify right))
     )
-    (property "Footprint" "MCP9701AT-E_TT:SOT-23-3" (at 110.49 91.44 0)
+    (property "Footprint" "BAT60JFILM:SOT-23-3" (at 110.49 91.44 0)
       (effects (font (size 1.524 1.524)) (justify left) hide)
     )
