File: Overall schematic/overall scematic/digi temp.kicad_sch (KiCad schematic)
At the start: 0 parts

Commit message: Add files via upload
Parts:
- added C?: 10n, symbol Device:C
- added R? (x2): 5k, symbol Device:R
- added SW?: SW_DIP_x01, symbol Switch:SW_DIP_x01
- added U?: TMP112AIDRLR, SOT50P160X60-6N, symbol TMP112AIDRLR:TMP112AIDRLR
Connections:
- new net: C?.1, R?.2, U?.5 (V+)
- new net Alert: R?.2, SW?.2, U?.3 (ALERT)
- new net GND: C?.2, SW?.1, U?.2 (GND), U?.4 (ADD0)
- new net PB12: U?.6 (SDA)
- new net SCL: U?.1 (SCL)
- new net Supply Voltage: R?.1, R?.1

Commit message: updated schematic
Connections:
- net PB12 renamed SDA
Changed lines of the file:
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@@
     (stroke (width 0) (type default))
-  )
-  (global_label "SCL" (shape output) (at 93.98 91.44 180) (fields_autoplaced)
-    (effects (font (size 1.27 1.27)) (justify right))
-    (property "Intersheetrefs" "${INTERSHEET_REFS}" (at 87.5666 91.44 0)
-      (effects (font (size 1.27 1.27)) (justify right) hide)
-    )
   )
   (global_label "Alert" (shape output) (at 187.96 93.98 0) (fields_autoplaced)
@@
     )
   )
-  (global_label "PB12" (shape output) (at 93.98 96.52 180) (fields_autoplaced)
+  (hierarchical_label "SCL" (shape input) (at 93.98 91.44 180) (fields_autoplaced)
     (effects (font (size 1.27 1.27)) (justify right))
-    (property "Intersheetrefs" "${INTERSHEET_REFS}" (at 86.1152 96.52 0)
-      (effects (font (size 1.27 1.27)) (justify right) hide)
-    )
   )
-  (global_label "Supply Voltage" (shape input) (at 165.1 64.77 90) (fields_autoplaced)
+  (hierarchical_label "Supply Voltage" (shape input) (at 165.1 64.77 90) (fields_autoplaced)
     (effects (font (size 1.27 1.27)) (justify left))
-    (property "Intersheetrefs" "${INTERSHEET_REFS}" (at 165.1 47.7978 90)
-      (effects (font (size 1.27 1.27)) (justify left) hide)
-    )
+  )
+  (hierarchical_label "SDA" (shape input) (at 93.98 96.52 180) (fields_autoplaced)
+    (effects (font (size 1.27 1.27)) (justify right))
   )
   (symbol (lib_id "Device:C") (at 165.1 86.36 0) (unit 1)

Commit message: Add files via upload
Parts:
- removed C?: 10n, symbol Device:C
- removed R? (x2): 5k, symbol Device:R
- removed SW?: SW_DIP_x01, symbol Switch:SW_DIP_x01
- removed U?: TMP112AIDRLR, SOT50P160X60-6N, symbol TMP112AIDRLR:TMP112AIDRLR
- added C5: CL21B104KCFNNNE, CAPC2012X140N, symbol CL21B104KCFNNNE:CL21B104KCFNNNE
- added U4: HDC1080, Package_SON:Texas_PWSON-N6, symbol Sensor_Humidity:HDC1080
Connections:
- net GND: now also C5.2, U4.2 (GND)
- new net Clock: U4.6 (SCL)
- new net Data: U4.1 (SDA)
- new net Vreg_Out: C5.1, U4.5 (VCC)

Commit message: fully annotated
Parts:
- C5: footprint CAPC2012X140N -> (none)
Connections:
- net Clock renamed SCL
- net Data renamed SDA
- net Vreg_Out renamed Supply_Voltage
Changed lines of the file:
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@@
     (stroke (width 0) (type default))
   )
-  (global_label "Data" (shape bidirectional) (at 175.26 92.71 0) (fields_autoplaced)
+  (hierarchical_label "Supply_Voltage" (shape input) (at 123.19 78.74 90) (fields_autoplaced)
     (effects (font (size 1.27 1.27)) (justify left))
-    (property "Intersheetrefs" "${INTERSHEET_REFS}" (at 183.5708 92.71 0)
-      (effects (font (size 1.27 1.27)) (justify left) hide)
-    )
   )
-  (global_label "Clock" (shape input) (at 175.26 90.17 0) (fields_autoplaced)
+  (hierarchical_label "SDA" (shape bidirectional) (at 175.26 92.71 0) (fields_autoplaced)
     (effects (font (size 1.27 1.27)) (justify left))
-    (property "Intersheetrefs" "${INTERSHEET_REFS}" (at 183.3667 90.17 0)
-      (effects (font (size 1.27 1.27)) (justify left) hide)
-    )
   )
-  (global_label "Vreg_Out" (shape input) (at 123.19 78.74 90) (fields_autoplaced)
+  (hierarchical_label "SCL" (shape input) (at 175.26 90.17 0) (fields_autoplaced)
     (effects (font (size 1.27 1.27)) (justify left))
-    (property "Intersheetrefs" "${INTERSHEET_REFS}" (at 123.19 67.549 90)
-      (effects (font (size 1.27 1.27)) (justify left) hide)
-    )
   )
   (symbol (lib_id "CL21B104KCFNNNE:CL21B104KCFNNNE") (at 123.19 93.98 90) (unit 1)
@@
       (effects (font (size 1.27 1.27)) (justify right))
     )
-    (property "Footprint" "CAPC2012X140N" (at 123.19 93.98 0)
+    (property "Footprint" "" (at 123.19 93.98 0)
       (effects (font (size 1.27 1.27)) (justify left bottom) hide)
     )
@@
   (symbol (lib_id "power:GND") (at 123.19 106.68 0) (unit 1)
     (in_bom yes) (on_board yes) (dnp no) (fields_autoplaced)
-    (property "Reference" "#PWR?" (at 123.19 113.03 0)
+    (property "Reference" "#PWR010" (at 123.19 113.03 0)
       (effects (font (size 1.27 1.27)) hide)
     )
@@
       (project "overall scematic"
         (path "/9230863d-68c5-4e85-a5d4-0f54ecfbae5b/8c854172-02c8-417f-bf92-0562f4d1bdee"
-          (reference "#PWR?") (unit 1)
+          (reference "#PWR010") (unit 1)
         )
       )

Commit message: updated everything
Parts:
- C5: footprint (none) -> CL21B104KCFNNNE:CAPC2012X140N
Changed lines of the file:
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@@
       (effects (font (size 1.27 1.27)) (justify right))
     )
-    (property "Footprint" "" (at 123.19 93.98 0)
+    (property "Footprint" "CL21B104KCFNNNE:CAPC2012X140N" (at 123.19 93.98 0)
       (effects (font (size 1.27 1.27)) (justify left bottom) hide)
     )

Commit message: BOM
Other:
- company: (none) -> University of capetown
- title: (none) -> 3088_group22_design
Changed lines of the file:
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@@
 (kicad_sch (version 20230121) (generator eeschema)
   (paper "A4")
+  (title_block
+    (title "3088_group22_design")
+    (date "2023-03-20")
+    (rev "3")
+    (company "University of capetown")
+  )
   (junction (at 123.19 100.33) (diameter 0) (color 0 0 0 0)
   )

Commit message: The final Gerber
Parts:
- renumbered U4 to U1
Changed lines of the file:
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@@
   (symbol (lib_id "Sensor_Humidity:HDC1080") (at 152.4 92.71 0) (unit 1)
     (in_bom yes) (on_board yes) (dnp no)
-    (property "Reference" "U4" (at 161.29 97.79 0)
+    (property "Reference" "U1" (at 161.29 97.79 0)
       (effects (font (size 1.27 1.27)) (justify right))
     )
@@
       (project "overall scematic"
         (path "/9230863d-68c5-4e85-a5d4-0f54ecfbae5b/8c854172-02c8-417f-bf92-0562f4d1bdee"
-          (reference "U4") (unit 1)
+          (reference "U1") (unit 1)
         )
       )
@@
   (symbol (lib_id "power:GND") (at 123.19 106.68 0) (unit 1)
     (in_bom yes) (on_board yes) (dnp no) (fields_autoplaced)
-    (property "Reference" "#PWR010" (at 123.19 113.03 0)
+    (property "Reference" "#PWR0102" (at 123.19 113.03 0)
       (effects (font (size 1.27 1.27)) hide)
     )
@@
       (project "overall scematic"
         (path "/9230863d-68c5-4e85-a5d4-0f54ecfbae5b/8c854172-02c8-417f-bf92-0562f4d1bdee"
-          (reference "#PWR010") (unit 1)
+          (reference "#PWR0102") (unit 1)
         )
       )
