File: Overall schematic/overall scematic/digi temp.kicad_sch (KiCad schematic)
At the start: 2 parts, among them U1 HDC1080

Commit message: hail mary
Parts:
- added R7, R8: 4.7k, Resistor_SMD:R_0805_2012Metric, symbol Device:R_US
- C5: footprint CL21B104KCFNNNE:CAPC2012X140N -> BAT60JFILM:CAPC2012X140N
- renumbered U1 to U2
Connections:
- net SCL: now also R8.2
- net SDA: now also R7.2
- net Supply_Voltage: now also R7.1, R8.1
Changed lines of the file:
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@@
     (company "University of capetown")
   )
+  (junction (at 123.19 73.66) (diameter 0) (color 0 0 0 0)
+  )
   (junction (at 123.19 100.33) (diameter 0) (color 0 0 0 0)
   )
+  (junction (at 172.72 90.17) (diameter 0) (color 0 0 0 0)
+  )
+  (junction (at 168.91 76.2) (diameter 0) (color 0 0 0 0)
+  )
   (junction (at 123.19 85.09) (diameter 0) (color 0 0 0 0)
   )
-  (wire (pts (xy 160.02 92.71) (xy 175.26 92.71))
+  (junction (at 163.83 92.71) (diameter 0) (color 0 0 0 0)
+  )
+  (wire (pts (xy 172.72 86.36) (xy 172.72 90.17))
+    (stroke (width 0) (type default))
+  )
+  (wire (pts (xy 123.19 73.66) (xy 123.19 85.09))
+    (stroke (width 0) (type default))
+  )
+  (wire (pts (xy 160.02 92.71) (xy 163.83 92.71))
+    (stroke (width 0) (type default))
+  )
+  (wire (pts (xy 172.72 90.17) (xy 175.26 90.17))
+    (stroke (width 0) (type default))
+  )
+  (wire (pts (xy 163.83 92.71) (xy 175.26 92.71))
+    (stroke (width 0) (type default))
+  )
+  (wire (pts (xy 172.72 78.74) (xy 172.72 76.2))
+    (stroke (width 0) (type default))
+  )
+  (wire (pts (xy 168.91 73.66) (xy 168.91 76.2))
+    (stroke (width 0) (type default))
+  )
+  (wire (pts (xy 172.72 76.2) (xy 168.91 76.2))
+    (stroke (width 0) (type default))
+  )
+  (wire (pts (xy 163.83 76.2) (xy 163.83 78.74))
     (stroke (width 0) (type default))
   )
@@
     (stroke (width 0) (type default))
   )
-  (wire (pts (xy 160.02 90.17) (xy 175.26 90.17))
+  (wire (pts (xy 160.02 90.17) (xy 172.72 90.17))
+    (stroke (width 0) (type default))
+  )
+  (wire (pts (xy 163.83 86.36) (xy 163.83 92.71))
+    (stroke (width 0) (type default))
+  )
+  (wire (pts (xy 123.19 73.66) (xy 168.91 73.66))
     (stroke (width 0) (type default))
   )
@@
     (stroke (width 0) (type default))
   )
-  (wire (pts (xy 123.19 78.74) (xy 123.19 85.09))
+  (wire (pts (xy 168.91 76.2) (xy 163.83 76.2))
+    (stroke (width 0) (type default))
+  )
+  (wire (pts (xy 123.19 69.85) (xy 123.19 73.66))
     (stroke (width 0) (type default))
   )
@@
     (stroke (width 0) (type default))
   )
-  (hierarchical_label "Supply_Voltage" (shape input) (at 123.19 78.74 90) (fields_autoplaced)
+  (hierarchical_label "Supply_Voltage" (shape input) (at 123.19 69.85 90) (fields_autoplaced)
     (effects (font (size 1.27 1.27)) (justify left))
   )
@@
     (effects (font (size 1.27 1.27)) (justify left))
   )
-  (hierarchical_label "SCL" (shape input) (at 175.26 90.17 0) (fields_autoplaced)
+  (hierarchical_label "SCL" (shape bidirectional) (at 175.26 90.17 0) (fields_autoplaced)
     (effects (font (size 1.27 1.27)) (justify left))
   )
@@
       (effects (font (size 1.27 1.27)) (justify right))
     )
-    (property "Footprint" "CL21B104KCFNNNE:CAPC2012X140N" (at 123.19 93.98 0)
+    (property "Footprint" "BAT60JFILM:CAPC2012X140N" (at 123.19 93.98 0)
       (effects (font (size 1.27 1.27)) (justify left bottom) hide)
     )
@@
   (symbol (lib_id "Sensor_Humidity:HDC1080") (at 152.4 92.71 0) (unit 1)
     (in_bom yes) (on_board yes) (dnp no)
-    (property "Reference" "U1" (at 161.29 97.79 0)
+    (property "Reference" "U2" (at 161.29 97.79 0)
       (effects (font (size 1.27 1.27)) (justify right))
     )
@@
       (project "overall scematic"
         (path "/9230863d-68c5-4e85-a5d4-0f54ecfbae5b/8c854172-02c8-417f-bf92-0562f4d1bdee"
-          (reference "U1") (unit 1)
-        )
-      )
+          (reference "U2") (unit 1)
+        )
+      )
+    )
+  )
+  (symbol (lib_id "Device:R_US") (at 163.83 82.55 0) (unit 1)
+    (in_bom yes) (on_board yes) (dnp no) (fields_autoplaced)
+    (property "Reference" "R7" (at 166.37 81.915 0)
+      (effects (font (size 1.27 1.27)) (justify left))
+    )
+    (property "Value" "4.7k" (at 166.37 84.455 0)
+      (effects (font (size 1.27 1.27)) (justify left))
+    )
+    (property "Footprint" "Resistor_SMD:R_0805_2012Metric" (at 164.846 82.804 90)
+      (effects (font (size 1.27 1.27)) hide)
+    )
+    (property "Datasheet" "~" (at 163.83 82.55 0)
+      (effects (font (size 1.27 1.27)) hide)
+    )
+    (pin "1")
+    (pin "2")
+    (instances
+      (project "overall scematic"
+        (path "/9230863d-68c5-4e85-a5d4-0f54ecfbae5b/8c854172-02c8-417f-bf92-0562f4d1bdee"
+          (reference "R7") (unit 1)
+        )
+      )
+    )
+  )
+  (symbol (lib_id "Device:R_US") (at 172.72 82.55 0) (unit 1)
+    (in_bom yes) (on_board yes) (dnp no) (fields_autoplaced)
+    (property "Reference" "R8" (at 175.26 81.915 0)
+      (effects (font (size 1.27 1.27)) (justify left))
+    )
+    (property "Value" "4.7k" (at 175.26 84.455 0)
+      (effects (font (size 1.27 1.27)) (justify left))
+    )
+    (property "Footprint" "Resistor_SMD:R_0805_2012Metric" (at 173.736 82.804 90)
+      (effects (font (size 1.27 1.27)) hide)
+    )
+    (property "Datasheet" "~" (at 172.72 82.55 0)
+      (effects (font (size 1.27 1.27)) hide)
+    )
+    (pin "1")
+    (pin "2")
+    (instances
+      (project "overall scematic"
+        (path "/9230863d-68c5-4e85-a5d4-0f54ecfbae5b/8c854172-02c8-417f-bf92-0562f4d1bdee"
+          (reference "R8") (unit 1)
+        )
+      )
