File: Overall schematic/overall scematic/overall scematic.kicad_pcb (KiCad board)
At the start: 2 copper layers, 100 x 100 mm, 45 parts, among them IC1 battery protection IC DW01A-G, J1 USB_B_Micro, J12 Conn_01x24_Socket, J13 Conn_01x24_Socket, J19 Conn_01x02_Pin, J2 Conn_01x02_Pin, J3 Battery Charger IC TP4056, J4 Conn_01x02_Pin, J5 Conn_01x02_Pin, J6 Conn_01x02_Pin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

Commit message: hail marry
Parts:
- removed J12, J13: Conn_01x24_Socket, BAT60JFILM:SAMTEC_SSQ-120-03-G-D
- moved J1 1.50 mm to (112.8, 132.4), turned to -90 degrees
Routing:
- net Data +: track 53.2 -> 11.9 mm
- net /Micro controller pin outs/PB12: track 37.9 -> 0.00 mm
- net /SCL: track 92.9 -> 61.4 mm
- net /Micro controller pin outs/PB14: track 26.6 -> 0.00 mm
- net /Micro controller pin outs/PA8: track 26.2 -> 0.00 mm, vias 1 -> 0
- net /Micro controller pin outs/PB13: track 25.5 -> 0.00 mm
- net /Micro controller pin outs/PA5: track 24.6 -> 0.00 mm
- net /SDA: track 75.8 -> 51.8 mm
- net /Micro controller pin outs/PB2: track 22.8 -> 0.00 mm
- net /Micro controller pin outs/PB15: track 21.7 -> 0.00 mm
- net /Micro controller pin outs/PB1: track 20.9 -> 0.00 mm
- net /Micro controller pin outs/PB0: track 20.2 -> 0.00 mm
- net /Micro controller pin outs/PA12: track 18.5 -> 0.00 mm
- net /Micro controller pin outs/PA7: track 17.7 -> 0.16 mm
- net /Micro controller pin outs/PA11: track 16.6 -> 0.00 mm
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Other:
- board text added: "Group_22"
- board text added: "Loic Kibambo Best Nkhumeleni Maisha Magavha"
