File: Overall schematic/overall scematic/overall scematic.kicad_pcb (KiCad board)
At the start: 2 copper layers, 100 x 100 mm, 43 parts, among them IC1 battery protection IC DW01A-G, J1 USB_B_Micro, J10 Conn_01x02_Pin, J19 Conn_01x02_Pin, J2 Conn_01x02_Pin, J3 Battery Charger IC TP4056, J4 Conn_01x02_Pin, J5 Conn_01x02_Pin, J6 Conn_01x02_Pin, J7 Conn_01x02_Pin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

Commit message: let the code begin
Parts:
- J19: value Conn_01x02_Pin -> C5116481
Other:
- board text added: "Thanks for 3088. This should be a 16 credit course"
Changed lines of the file:
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@@
         (effects (font (size 1 1) (thickness 0.15)))
     )
-    (fp_text value "Conn_01x02_Pin" (at 1.075 5.17) (layer "F.Fab")
+    (fp_text value "C5116481" (at 1.075 5.17) (layer "F.Fab")
         (effects (font (size 1 1) (thickness 0.15)))
     )
@@
     (property "ki_description" "Light emitting diode")
     (property "ki_keywords" "LED diode")
-    (attr smd)
+    (attr smd exclude_from_pos_files exclude_from_bom)
     (fp_text reference "D1" (at 0 -1.65) (layer "F.SilkS")
         (effects (font (size 1 1) (thickness 0.15)))
@@
     (property "ki_keywords" "R res resistor")
     (attr through_hole exclude_from_pos_files exclude_from_bom)
-    (fp_text reference "R3" (at 2.54 -2.37) (layer "F.SilkS")
+    (fp_text reference "R3" (at 0 0) (layer "F.SilkS")
         (effects (font (size 1 1) (thickness 0.15)))
     )
@@
   (gr_rect (start 110 52) (end 210 152)
     (stroke (width 0.1) (type default)) (fill none) (layer "Edge.Cuts"))
+  (gr_text "Thanks for 3088.\nThis should be a 16 \ncredit course" (at 207 130.5 90) (layer "F.Cu")
+    (effects (font (size 1.5 1.5) (thickness 0.3) bold) (justify left bottom))
+  )
   (gr_text "Loic Kibambo\nBest Nkhumeleni\nMaisha Magavha\n" (at 200.5 99 90) (layer "F.Cu")
     (effects (font (size 1.5 1.5) (thickness 0.3) bold) (justify left bottom))
