File: Overall schematic/overall scematic/_autosave-overall scematic.kicad_pcb (KiCad board)
At the start: 2 copper layers, 100 x 100 mm, 43 parts, among them IC1 battery protection IC DW01A-G, J1 USB_B_Micro, J10 Conn_01x02_Pin, J19 Conn_01x02_Pin, J2 Conn_01x02_Pin, J3 Battery Charger IC TP4056, J4 Conn_01x02_Pin, J5 Conn_01x02_Pin, J6 Conn_01x02_Pin, J7 Conn_01x02_Pin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

Commit message: the j's
Parts:
- J19: value Conn_01x02_Pin -> C5116481
Changed lines of the file:
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@@
     (property "ki_description" "test point")
     (property "ki_keywords" "test point tp")
-    (attr exclude_from_pos_files exclude_from_bom)
+    (attr exclude_from_pos_files)
     (fp_text reference "TP3" (at 1.3 -2) (layer "F.SilkS")
         (effects (font (size 1 1) (thickness 0.15)))
@@
     (property "ki_description" "Resistor")
     (property "ki_keywords" "R res resistor")
-    (attr through_hole exclude_from_pos_files exclude_from_bom)
+    (attr through_hole exclude_from_pos_files)
     (fp_text reference "R5" (at 2.54 -2.37) (layer "F.SilkS")
         (effects (font (size 1 1) (thickness 0.15)))
@@
         (effects (font (size 1 1) (thickness 0.15)))
     )
-    (fp_text value "Conn_01x02_Pin" (at 1.075 5.17) (layer "F.Fab")
+    (fp_text value "C5116481" (at 1.075 5.17) (layer "F.Fab")
         (effects (font (size 1 1) (thickness 0.15)))
     )
@@
     (property "ki_description" "Single-cell battery")
     (property "ki_keywords" "battery cell")
-    (attr smd exclude_from_pos_files exclude_from_bom)
+    (attr smd exclude_from_pos_files)
     (fp_text reference "BT1" (at 0 -0.5 unlocked) (layer "F.SilkS")
         (effects (font (size 1 1) (thickness 0.15)))
@@
     (property "ki_description" "test point")
     (property "ki_keywords" "test point tp")
-    (attr exclude_from_pos_files exclude_from_bom)
+    (attr exclude_from_pos_files)
     (fp_text reference "TP1" (at 1.3 -2) (layer "F.SilkS")
         (effects (font (size 1 1) (thickness 0.15)))
@@
     (property "ki_description" "Resistor")
     (property "ki_keywords" "R res resistor")
-    (attr through_hole exclude_from_pos_files exclude_from_bom)
+    (attr through_hole exclude_from_pos_files)
     (fp_text reference "R4" (at 2.54 -2.37) (layer "F.SilkS")
         (effects (font (size 1 1) (thickness 0.15)))
@@
     (property "ki_description" "Resistor")
     (property "ki_keywords" "R res resistor")
-    (attr through_hole exclude_from_pos_files exclude_from_bom)
+    (attr through_hole exclude_from_pos_files)
     (fp_text reference "R6" (at 2.54 -2.37) (layer "F.SilkS")
         (effects (font (size 1 1) (thickness 0.15)))
@@
     (property "Sheetfile" "micro controlter interface.kicad_sch")
     (property "Sheetname" "Micro controller pin outs")
-    (attr through_hole exclude_from_pos_files exclude_from_bom)
+    (attr through_hole exclude_from_pos_files)
     (fp_text reference "U3" (at -0.31 -0.16 90 unlocked) (layer "F.SilkS")
         (effects (font (size 1 1) (thickness 0.15)))
@@
     (property "ki_description" "test point")
     (property "ki_keywords" "test point tp")
-    (attr exclude_from_pos_files exclude_from_bom)
+    (attr exclude_from_pos_files)
     (fp_text reference "TP2" (at 1.3 -2) (layer "F.SilkS")
         (effects (font (size 1 1) (thickness 0.15)))
@@
     (property "ki_description" "Resistor")
     (property "ki_keywords" "R res resistor")
-    (attr through_hole exclude_from_pos_files exclude_from_bom)
+    (attr through_hole exclude_from_pos_files)
     (fp_text reference "R1" (at 5.08 -2.37) (layer "F.SilkS")
         (effects (font (size 1 1) (thickness 0.15)))
@@
     (property "ki_description" "Generic connector, double row, 02x24, counter clockwise pin numbering scheme (similar to DIP package numbering), script generated (kicad-library-utils/schlib/autogen/connector/)")
     (property "ki_keywords" "connector")
-    (attr smd exclude_from_pos_files exclude_from_bom)
+    (attr smd exclude_from_pos_files)
     (fp_text reference "J9" (at -0.2 -6.1 -90 unlocked) (layer "F.SilkS") hide
         (effects (font (size 1 1) (thickness 0.15)))
@@
     (property "ki_description" "Resistor")
     (property "ki_keywords" "R res resistor")
-    (attr through_hole exclude_from_pos_files exclude_from_bom)
+    (attr through_hole exclude_from_pos_files)
     (fp_text reference "R3" (at 2.54 -2.37) (layer "F.SilkS")
         (effects (font (size 1 1) (thickness 0.15)))
