File: Overall schematic/overall scematic/micro controlter interface.kicad_sch (KiCad schematic)
At the start: 4 parts, among them J1 DB25_Receptacle, J2 DB25_Receptacle, U1 AT24CS01-STUM, U2 STM32F030R8Tx

Commit message: Add files via upload
Parts:
- renumbered J2 to J?, J1 to J?, U2 to U?, U1 to U?
Changed lines of the file:
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@@
   (symbol (lib_id "power:GND") (at 156.21 111.76 0) (unit 1)
     (in_bom yes) (on_board yes) (dnp no) (fields_autoplaced)
-    (property "Reference" "#PWR03" (at 156.21 118.11 0)
+    (property "Reference" "#PWR?" (at 156.21 118.11 0)
       (effects (font (size 1.27 1.27)) hide)
     )
@@
       (project "overall scematic"
         (path "/9230863d-68c5-4e85-a5d4-0f54ecfbae5b/8d35112e-3dcb-4f8a-ab75-188a6b3d82be"
-          (reference "#PWR03") (unit 1)
+          (reference "#PWR?") (unit 1)
         )
       )
@@
   (symbol (lib_id "power:GND") (at 242.57 50.8 180) (unit 1)
     (in_bom yes) (on_board yes) (dnp no) (fields_autoplaced)
-    (property "Reference" "#PWR05" (at 242.57 44.45 0)
+    (property "Reference" "#PWR?" (at 242.57 44.45 0)
       (effects (font (size 1.27 1.27)) hide)
     )
@@
       (project "overall scematic"
         (path "/9230863d-68c5-4e85-a5d4-0f54ecfbae5b/8d35112e-3dcb-4f8a-ab75-188a6b3d82be"
-          (reference "#PWR05") (unit 1)
+          (reference "#PWR?") (unit 1)
         )
       )
@@
   (symbol (lib_id "MCU_ST_STM32F0:STM32F030R8Tx") (at 171.45 83.82 0) (unit 1)
     (in_bom yes) (on_board yes) (dnp no) (fields_autoplaced)
-    (property "Reference" "U2" (at 175.9459 129.54 0)
+    (property "Reference" "U?" (at 175.9459 129.54 0)
       (effects (font (size 1.27 1.27)) (justify left))
     )
@@
       (project "overall scematic"
         (path "/9230863d-68c5-4e85-a5d4-0f54ecfbae5b/8d35112e-3dcb-4f8a-ab75-188a6b3d82be"
-          (reference "U2") (unit 1)
+          (reference "U?") (unit 1)
         )
       )
@@
   (symbol (lib_id "Custom spi connector:DB25_Receptacle") (at 77.47 81.28 180) (unit 1)
     (in_bom yes) (on_board yes) (dnp no) (fields_autoplaced)
-    (property "Reference" "J2" (at 77.47 43.18 0)
+    (property "Reference" "J?" (at 77.47 43.18 0)
       (effects (font (size 1.27 1.27)))
     )
@@
       (project "overall scematic"
         (path "/9230863d-68c5-4e85-a5d4-0f54ecfbae5b/8d35112e-3dcb-4f8a-ab75-188a6b3d82be"
-          (reference "J2") (unit 1)
+          (reference "J?") (unit 1)
         )
       )
@@
   (symbol (lib_id "power:GND") (at 152.4 43.18 180) (unit 1)
     (in_bom yes) (on_board yes) (dnp no) (fields_autoplaced)
-    (property "Reference" "#PWR08" (at 152.4 36.83 0)
+    (property "Reference" "#PWR?" (at 152.4 36.83 0)
       (effects (font (size 1.27 1.27)) hide)
     )
@@
       (project "overall scematic"
         (path "/9230863d-68c5-4e85-a5d4-0f54ecfbae5b/8d35112e-3dcb-4f8a-ab75-188a6b3d82be"
-          (reference "#PWR08") (unit 1)
+          (reference "#PWR?") (unit 1)
         )
       )
@@
   (symbol (lib_id "power:PWR_FLAG") (at 219.71 34.29 0) (unit 1)
     (in_bom yes) (on_board yes) (dnp no) (fields_autoplaced)
-    (property "Reference" "#FLG02" (at 219.71 32.385 0)
+    (property "Reference" "#FLG?" (at 219.71 32.385 0)
       (effects (font (size 1.27 1.27)) hide)
     )
@@
       (project "overall scematic"
         (path "/9230863d-68c5-4e85-a5d4-0f54ecfbae5b/8d35112e-3dcb-4f8a-ab75-188a6b3d82be"
-          (reference "#FLG02") (unit 1)
+          (reference "#FLG?") (unit 1)
         )
       )
@@
   (symbol (lib_id "power:GND") (at 92.71 111.76 0) (unit 1)
     (in_bom yes) (on_board yes) (dnp no) (fields_autoplaced)
-    (property "Reference" "#PWR02" (at 92.71 118.11 0)
+    (property "Reference" "#PWR?" (at 92.71 118.11 0)
       (effects (font (size 1.27 1.27)) hide)
     )
@@
       (project "overall scematic"
         (path "/9230863d-68c5-4e85-a5d4-0f54ecfbae5b/8d35112e-3dcb-4f8a-ab75-188a6b3d82be"
-          (reference "#PWR02") (unit 1)
+          (reference "#PWR?") (unit 1)
         )
       )
@@
   (symbol (lib_id "power:GND") (at 125.73 57.15 0) (unit 1)
     (in_bom yes) (on_board yes) (dnp no) (fields_autoplaced)
-    (property "Reference" "#PWR06" (at 125.73 63.5 0)
+    (property "Reference" "#PWR?" (at 125.73 63.5 0)
       (effects (font (size 1.27 1.27)) hide)
     )
@@
       (project "overall scematic"
         (path "/9230863d-68c5-4e85-a5d4-0f54ecfbae5b/8d35112e-3dcb-4f8a-ab75-188a6b3d82be"
-          (reference "#PWR06") (unit 1)
+          (reference "#PWR?") (unit 1)
         )
       )
@@
   (symbol (lib_id "power:GND") (at 190.5 43.18 180) (unit 1)
     (in_bom yes) (on_board yes) (dnp no) (fields_autoplaced)
-    (property "Reference" "#PWR07" (at 190.5 36.83 0)
+    (property "Reference" "#PWR?" (at 190.5 36.83 0)
       (effects (font (size 1.27 1.27)) hide)
     )
@@
       (project "overall scematic"
         (path "/9230863d-68c5-4e85-a5d4-0f54ecfbae5b/8d35112e-3dcb-4f8a-ab75-188a6b3d82be"
-          (reference "#PWR07") (unit 1)
+          (reference "#PWR?") (unit 1)
         )
       )
@@
   (symbol (lib_id "power:+5V") (at 210.82 34.29 0) (unit 1)
     (in_bom yes) (on_board yes) (dnp no) (fields_autoplaced)
-    (property "Reference" "#PWR04" (at 210.82 38.1 0)
+    (property "Reference" "#PWR?" (at 210.82 38.1 0)
       (effects (font (size 1.27 1.27)) hide)
     )
@@
       (project "overall scematic"
         (path "/9230863d-68c5-4e85-a5d4-0f54ecfbae5b/8d35112e-3dcb-4f8a-ab75-188a6b3d82be"
-          (reference "#PWR04") (unit 1)
+          (reference "#PWR?") (unit 1)
         )
       )
@@
   (symbol (lib_id "Memory_EEPROM:AT24CS01-STUM") (at 124.46 49.53 0) (unit 1)
     (in_bom yes) (on_board yes) (dnp no) (fields_autoplaced)
-    (property "Reference" "U1" (at 115.57 48.895 0)
+    (property "Reference" "U?" (at 115.57 48.895 0)
       (effects (font (size 1.27 1.27)) (justify right))
     )
@@
       (project "overall scematic"
         (path "/9230863d-68c5-4e85-a5d4-0f54ecfbae5b/8d35112e-3dcb-4f8a-ab75-188a6b3d82be"
-          (reference "U1") (unit 1)
+          (reference "U?") (unit 1)
         )
       )
@@
   (symbol (lib_id "Custom spi connector:DB25_Receptacle") (at 254 91.44 0) (unit 1)
     (in_bom yes) (on_board yes) (dnp no) (fields_autoplaced)
-    (property "Reference" "J1" (at 259.08 90.805 0)
+    (property "Reference" "J?" (at 259.08 90.805 0)
       (effects (font (size 1.27 1.27)) (justify left))
     )
@@
       (project "overall scematic"
         (path "/9230863d-68c5-4e85-a5d4-0f54ecfbae5b/8d35112e-3dcb-4f8a-ab75-188a6b3d82be"
-          (reference "J1") (unit 1)
+          (reference "J?") (unit 1)
         )
       )
@@
   (symbol (lib_id "power:+3.3V") (at 127 34.29 0) (unit 1)
     (in_bom yes) (on_board yes) (dnp no) (fields_autoplaced)
-    (property "Reference" "#PWR01" (at 127 38.1 0)
+    (property "Reference" "#PWR?" (at 127 38.1 0)
       (effects (font (size 1.27 1.27)) hide)
     )
@@
       (project "overall scematic"
         (path "/9230863d-68c5-4e85-a5d4-0f54ecfbae5b/8d35112e-3dcb-4f8a-ab75-188a6b3d82be"
-          (reference "#PWR01") (unit 1)
+          (reference "#PWR?") (unit 1)
         )
       )
@@
   (symbol (lib_id "power:PWR_FLAG") (at 116.84 34.29 0) (unit 1)
     (in_bom yes) (on_board yes) (dnp no) (fields_autoplaced)
-    (property "Reference" "#FLG01" (at 116.84 32.385 0)
+    (property "Reference" "#FLG?" (at 116.84 32.385 0)
       (effects (font (size 1.27 1.27)) hide)
     )
@@
       (project "overall scematic"
         (path "/9230863d-68c5-4e85-a5d4-0f54ecfbae5b/8d35112e-3dcb-4f8a-ab75-188a6b3d82be"
-          (reference "#FLG01") (unit 1)
-        )
-      )
+          (reference "#FLG?") (unit 1)
+        )
+      )

Commit message: fully annotated
Parts:
- removed U?: STM32F030R8Tx, Package_QFP:LQFP-64_10x10mm_P0.5mm, symbol MCU_ST_STM32F0:STM32F030R8Tx
- gave numbers to parts that had none: 3
Connections:
- net DAC line is gone; now on net GND: J9.13
- net I2C2 is gone; now on net I2C: J9.12
- net SPI2 is gone; now on net SPI: J8.15 (P15)
- net GND: no longer J8.16 (P16)
- net SCL: now reaches U2.1 (SCL)
- net SCL: now also J8.16 (P16)
- net I2C1 renamed I2C
- net SPI1 renamed SPI
- net data line gpio output renamed SDA
Other:
- note removed: "This is a similation of the stm 32 and her pins"

Commit message: updated everything
Parts:
- J8, J9: footprint (none) -> SSQ-120-03-G-D:SAMTEC_SSQ-120-03-G-D
Connections:
- net GND: no longer J8.14 (P14)
- net +3.3V renamed Supply_Voltage
- net I2C renamed I2C1
- net I2C1: no longer J9.12
- new net ADC: J8.14 (P14)
- new net I2C2: J9.12
Changed lines of the file:
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@@
   (junction (at 242.57 99.06) (diameter 0) (color 0 0 0 0)
   )
-  (junction (at 124.46 34.29) (diameter 0) (color 0 0 0 0)
-  )
   (junction (at 242.57 71.12) (diameter 0) (color 0 0 0 0)
   )
@@
   (junction (at 88.9 76.2) (diameter 0) (color 0 0 0 0)
   )
-  (junction (at 88.9 109.22) (diameter 0) (color 0 0 0 0)
-  )
   (junction (at 242.57 101.6) (diameter 0) (color 0 0 0 0)
   )
@@
   (junction (at 88.9 106.68) (diameter 0) (color 0 0 0 0)
   )
-  (junction (at 125.73 57.15) (diameter 0) (color 0 0 0 0)
-  )
   (junction (at 88.9 83.82) (diameter 0) (color 0 0 0 0)
   )
@@
     (stroke (width 0) (type default))
   )
-  (wire (pts (xy 125.73 57.15) (xy 124.46 57.15))
-    (stroke (width 0) (type default))
-  )
-  (wire (pts (xy 116.84 34.29) (xy 124.46 34.29))
-    (stroke (width 0) (type default))
-  )
   (wire (pts (xy 242.57 121.92) (xy 246.38 121.92))
     (stroke (width 0) (type default))
@@
     (stroke (width 0) (type default))
   )
-  (wire (pts (xy 88.9 109.22) (xy 156.21 109.22))
-    (stroke (width 0) (type default))
-  )
   (wire (pts (xy 88.9 91.44) (xy 88.9 88.9))
     (stroke (width 0) (type default))
@@
     (stroke (width 0) (type default))
   )
+  (wire (pts (xy 124.46 57.15) (xy 128.27 57.15))
+    (stroke (width 0) (type default))
+  )
   (wire (pts (xy 246.38 76.2) (xy 242.57 76.2))
     (stroke (width 0) (type default))
@@
     (stroke (width 0) (type default))
   )
-  (wire (pts (xy 88.9 106.68) (xy 88.9 109.22))
+  (wire (pts (xy 88.9 106.68) (xy 88.9 111.76))
     (stroke (width 0) (type default))
   )
@@
     (stroke (width 0) (type default))
   )
-  (wire (pts (xy 85.09 109.22) (xy 88.9 109.22))
+  (wire (pts (xy 85.09 109.22) (xy 156.21 109.22))
     (stroke (width 0) (type default))
   )
@@
     (stroke (width 0) (type default))
   )
-  (wire (pts (xy 134.62 57.15) (xy 125.73 57.15))
-    (stroke (width 0) (type default))
-  )
   (wire (pts (xy 88.9 76.2) (xy 88.9 73.66))
-    (stroke (width 0) (type default))
-  )
-  (wire (pts (xy 88.9 109.22) (xy 88.9 111.76))
     (stroke (width 0) (type default))
   )
@@
     )
   )
-  (global_label "I2C" (shape bidirectional) (at 186.69 114.3 180) (fields_autoplaced)
+  (global_label "I2C1" (shape bidirectional) (at 186.69 114.3 180) (fields_autoplaced)
     (effects (font (size 1.27 1.27)) (justify right))
-    (property "Intersheetrefs" "${INTERSHEET_REFS}" (at 179.5886 114.3 0)
+    (property "Intersheetrefs" "${INTERSHEET_REFS}" (at 178.3791 114.3 0)
       (effects (font (size 1.27 1.27)) (justify right) hide)
     )
@@
     )
   )
-  (global_label "I2C" (shape bidirectional) (at 186.69 116.84 180) (fields_autoplaced)
+  (global_label "I2C2" (shape bidirectional) (at 186.69 116.84 180) (fields_autoplaced)
     (effects (font (size 1.27 1.27)) (justify right))
-    (property "Intersheetrefs" "${INTERSHEET_REFS}" (at 179.5886 116.84 0)
+    (property "Intersheetrefs" "${INTERSHEET_REFS}" (at 178.3791 116.84 0)
       (effects (font (size 1.27 1.27)) (justify right) hide)
     )
@@
   )
   (hierarchical_label "SDA" (shape bidirectional) (at 135.89 46.99 0) (fields_autoplaced)
+    (effects (font (size 1.27 1.27)) (justify left))
+  )
+  (hierarchical_label "Supply_Voltage" (shape input) (at 127 34.29 90) (fields_autoplaced)
     (effects (font (size 1.27 1.27)) (justify left))
   )
@@
       (effects (font (size 1.27 1.27)))
     )
-    (property "Footprint" "" (at 77.47 81.28 0)
+    (property "Footprint" "SSQ-120-03-G-D:SAMTEC_SSQ-120-03-G-D" (at 77.47 81.28 0)
       (effects (font (size 1.27 1.27)) hide)
     )
@@
     )
   )
-  (symbol (lib_id "power:GND") (at 125.73 57.15 0) (unit 1)
+  (symbol (lib_id "power:GND") (at 134.62 57.15 0) (unit 1)
     (in_bom yes) (on_board yes) (dnp no) (fields_autoplaced)
-    (property "Reference" "#PWR013" (at 125.73 63.5 0)
-      (effects (font (size 1.27 1.27)) hide)
-    )
-    (property "Value" "GND" (at 125.73 62.23 0)
+    (property "Reference" "#PWR09" (at 134.62 63.5 0)
+      (effects (font (size 1.27 1.27)) hide)
+    )
+    (property "Value" "GND" (at 134.62 62.23 0)
       (effects (font (size 1.27 1.27)))
     )
-    (property "Footprint" "" (at 125.73 57.15 0)
-      (effects (font (size 1.27 1.27)) hide)
-    )
-    (property "Datasheet" "" (at 125.73 57.15 0)
+    (property "Footprint" "" (at 134.62 57.15 0)
+      (effects (font (size 1.27 1.27)) hide)
+    )
+    (property "Datasheet" "" (at 134.62 57.15 0)
       (effects (font (size 1.27 1.27)) hide)
     )
@@
     (instances
       (project "overall scematic"
+        (path "/9230863d-68c5-4e85-a5d4-0f54ecfbae5b/c494e013-0c38-49c8-84da-4f33138ae19d"
+          (reference "#PWR09") (unit 1)
+        )
         (path "/9230863d-68c5-4e85-a5d4-0f54ecfbae5b/8d35112e-3dcb-4f8a-ab75-188a6b3d82be"
-          (reference "#PWR013") (unit 1)
+          (reference "#PWR07") (unit 1)
+        )
+      )
+      (project "analogue_temparature"
+        (path "/fd616d34-a44b-4530-b77b-84bccfccd64d"
+          (reference "#PWR?") (unit 1)
+        )
+      )
+    )
+  )
+  (symbol (lib_id "power:GND") (at 128.27 57.15 0) (unit 1)
+    (in_bom yes) (on_board yes) (dnp no) (fields_autoplaced)
+    (property "Reference" "#PWR09" (at 128.27 63.5 0)
+      (effects (font (size 1.27 1.27)) hide)
+    )
+    (property "Value" "GND" (at 128.27 62.23 0)
+      (effects (font (size 1.27 1.27)))
+    )
+    (property "Footprint" "" (at 128.27 57.15 0)
+      (effects (font (size 1.27 1.27)) hide)
+    )
+    (property "Datasheet" "" (at 128.27 57.15 0)
+      (effects (font (size 1.27 1.27)) hide)
+    )
+    (pin "1")
+    (instances
+      (project "overall scematic"
+        (path "/9230863d-68c5-4e85-a5d4-0f54ecfbae5b/c494e013-0c38-49c8-84da-4f33138ae19d"
+          (reference "#PWR09") (unit 1)
+        )
+        (path "/9230863d-68c5-4e85-a5d4-0f54ecfbae5b/8d35112e-3dcb-4f8a-ab75-188a6b3d82be"
+          (reference "#PWR06") (unit 1)
+        )
+      )
+      (project "analogue_temparature"
+        (path "/fd616d34-a44b-4530-b77b-84bccfccd64d"
+          (reference "#PWR?") (unit 1)
         )
       )
@@
       (effects (font (size 1.27 1.27)) (justify left))
     )
-    (property "Footprint" "" (at 254 91.44 0)
+    (property "Footprint" "SSQ-120-03-G-D:SAMTEC_SSQ-120-03-G-D" (at 254 91.44 0)
       (effects (font (size 1.27 1.27)) hide)
     )
@@
         )
       )
-    )
-  )
-  (symbol (lib_id "power:+3.3V") (at 127 34.29 0) (unit 1)
-    (in_bom yes) (on_board yes) (dnp no) (fields_autoplaced)
-    (property "Reference" "#PWR014" (at 127 38.1 0)
-      (effects (font (size 1.27 1.27)) hide)
-    )
-    (property "Value" "+3.3V" (at 127 30.48 0)
-      (effects (font (size 1.27 1.27)))
-    )
-    (property "Footprint" "" (at 127 34.29 0)
-      (effects (font (size 1.27 1.27)) hide)
-    )
-    (property "Datasheet" "" (at 127 34.29 0)
-      (effects (font (size 1.27 1.27)) hide)
-    )
-    (pin "1")
-    (instances
-      (project "overall scematic"
-        (path "/9230863d-68c5-4e85-a5d4-0f54ecfbae5b/8d35112e-3dcb-4f8a-ab75-188a6b3d82be"
-          (reference "#PWR014") (unit 1)
-        )
-      )
-    )
-  )
-  (symbol (lib_id "power:PWR_FLAG") (at 116.84 34.29 0) (unit 1)
-    (in_bom yes) (on_board yes) (dnp no) (fields_autoplaced)
-    (property "Reference" "#FLG08" (at 116.84 32.385 0)
-      (effects (font (size 1.27 1.27)) hide)
-    )
-    (property "Value" "PWR_FLAG" (at 116.84 30.48 0)
-      (effects (font (size 1.27 1.27)))
-    )
-    (property "Footprint" "" (at 116.84 34.29 0)
-      (effects (font (size 1.27 1.27)) hide)
-    )
-    (property "Datasheet" "~" (at 116.84 34.29 0)
-      (effects (font (size 1.27 1.27)) hide)
-    )
-    (pin "1")
-    (instances
-      (project "overall scematic"
-        (path "/9230863d-68c5-4e85-a5d4-0f54ecfbae5b/8d35112e-3dcb-4f8a-ab75-188a6b3d82be"
-          (reference "#FLG08") (unit 1)
-        )
-      )

Commit message: BOM
Other:
- company: (none) -> University of capetown
- title: (none) -> 3088_group22_design
Changed lines of the file:
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@@
 (kicad_sch (version 20230121) (generator eeschema)
   (paper "A4")
+  (title_block
+    (title "3088_group22_design")
+    (date "2023-03-20")
+    (rev "3")
+    (company "University of capetown")
+  )
   (junction (at 242.57 81.28) (diameter 0) (color 0 0 0 0)
   )

Commit message: The final Gerber
Parts:
- added J10: Conn_01x09_Pin, Connector_PinHeader_2.54mm:PinHeader_1x03_P2.54mm_Vertical, symbol Connector:Conn_01x09_Pin
- added U3: STLINK_UCT, Module:ST_Morpho_Connector_144_STLink, symbol UCT:STLINK_UCT
- renumbered U2 to U4
Connections:
- net SPI is gone; now on net GND: J8.15 (P15), J8.3
- net USART1 is gone; now on net GND: J9.23 (P23)
- net USART2 is gone; now on net GND: J9.11
- net GND: now also J10.5 (Pin_5), U3.5 (GND); no longer J8.10, J8.12, J8.13, J8.25 (P25)
- net I2C1: now also U3.7 (T_SWCLK)
- net I2C2: now also U3.8 (T_SWDIO)
- net Supply_Voltage: now also J10.1 (Pin_1), J10.2 (Pin_2), U3.2 (V_Target)
- net ADC renamed Analogue_out
- new net Data +: J10.3 (Pin_3), U3.4 (USB_DP)
- new net Data -: J10.4 (Pin_4), U3.3 (USB_DM)
- new net NRST: J10.6 (Pin_6), J8.10, U3.6 (T_NRST)
- new net PA0: J10.9 (Pin_9), J8.13
- new net PB6: J10.7 (Pin_7), J8.12
- new net PB7: J10.8 (Pin_8), J8.25 (P25)
- new net Vreg_Out: U3.1 (5V_USB)
- no-connect marks 0 -> 1

Commit message: hail mary
Parts:
- removed J10: Conn_01x09_Pin, Connector_PinHeader_2.54mm:PinHeader_1x03_P2.54mm_Vertical, symbol Connector:Conn_01x09_Pin
- removed J8, J9: DB25_Receptacle, SSQ-120-03-G-D:SAMTEC_SSQ-120-03-G-D, symbol Custom spi connector:DB25_Receptacle
- added C1: 10nF, Capacitor_SMD:C_1206_3216Metric, symbol Device:C
- added J1, J2: Conn_01x24_Socket, BAT60JFILM:SAMTEC_SSQ-120-03-G-D, symbol Connector:Conn_01x24_Socket
- added J8: Conn_01x02_Pin, Connector_PinHeader_2.54mm:PinHeader_1x02_P2.54mm_Vertical, symbol Connector:Conn_01x02_Pin
- added J9: Conn_02x24_Counter_Clockwise, BAT60JFILM:STM32F051C6T6, symbol Connector_Generic:Conn_02x24_Counter_Clockwise
- added R1: 10k, Resistor_SMD:R_0805_2012Metric, symbol Device:R_Small_US
- added R4, R5: 1k, Resistor_SMD:R_0603_1608Metric, symbol Device:R_Small_US
- added SW1: SW_Push, Button_Switch_THT:SW_PUSH_6mm, symbol Switch:SW_Push
- U3: footprint Module:ST_Morpho_Connector_144_STLink -> BAT60JFILM:STLINK_UCT
Connections:
- net Analogue_out: now also J1.10 (Pin_10), J9.10 (Pin_10)
- net GND: now also C1.2, J1.23 (Pin_23), J1.8 (Pin_8), J2.2 (Pin_2), J9.23 (Pin_23), J9.47 (Pin_47), J9.8 (Pin_8), R1.1, SW1.1
- net NRST: now also J1.7 (Pin_7), J9.7 (Pin_7), SW1.2
- net PB6: now also U4.1 (SCL), J2.7 (Pin_7), J9.42 (Pin_42), R5.2
- net PB7: now also U4.3 (SDA), J2.6 (Pin_6), J9.43 (Pin_43), R4.2
- net SCL: now also J1.21 (Pin_21), J9.21 (Pin_21); no longer U4.1 (SCL)
- net SDA: now also J1.22 (Pin_22), J9.22 (Pin_22); no longer U4.3 (SDA)
- net Supply_Voltage: now also J1.24 (Pin_24), J2.1 (Pin_1), J8.2 (Pin_2), J9.24 (Pin_24), J9.48 (Pin_48), R4.1, R5.1; no longer U4.4 (VCC)
- net Vreg_Out: now also J1.1 (Pin_1), J9.1 (Pin_1)
- net I2C1 renamed PA9
- net PA9: now also J2.19 (Pin_19), J9.30 (Pin_30)
- net I2C2 renamed PA10
- net PA10: now also J2.18 (Pin_18), J9.31 (Pin_31)
- new net: C1.1, J8.1 (Pin_1), U4.4 (VCC)
- new net BOOT: J2.5 (Pin_5), J9.44 (Pin_44), R1.2
- new net PA1: J1.11 (Pin_11), J9.11 (Pin_11)
- new net PA11: J2.17 (Pin_17), J9.32 (Pin_32)
- new net PA12: J2.16 (Pin_16), J9.33 (Pin_33)
- new net PA13: J2.15 (Pin_15), J9.34 (Pin_34)
- new net PA14: J2.12 (Pin_12), J9.37 (Pin_37)
- new net PA15: J2.11 (Pin_11), J9.38 (Pin_38)
- new net PA2: J1.12 (Pin_12), J9.12 (Pin_12)
- new net PA3: J1.13 (Pin_13), J9.13 (Pin_13)
- new net PA4: J1.14 (Pin_14), J9.14 (Pin_14)
- new net PA5: J1.15 (Pin_15), J9.15 (Pin_15)
- new net PA6: J1.16 (Pin_16), J9.16 (Pin_16)
- new net PA7: J1.17 (Pin_17), J9.17 (Pin_17)
- new net PA8: J2.20 (Pin_20), J9.29 (Pin_29)
- new net PB0: J1.18 (Pin_18), J9.18 (Pin_18)
- new net PB1: J1.19 (Pin_19), J9.19 (Pin_19)
- new net PB12: J2.24 (Pin_24), J9.25 (Pin_25)
- new net PB13: J2.23 (Pin_23), J9.26 (Pin_26)
- new net PB14: J2.22 (Pin_22), J9.27 (Pin_27)
- new net PB15: J2.21 (Pin_21), J9.28 (Pin_28)
- new net PB2: J1.20 (Pin_20), J9.20 (Pin_20)
- new net PB3: J2.10 (Pin_10), J9.39 (Pin_39)
- new net PB4: J2.9 (Pin_9), J9.40 (Pin_40)
- new net PB5: J2.8 (Pin_8), J9.41 (Pin_41)
- new net PB8: J2.4 (Pin_4), J9.45 (Pin_45)
- new net PB9: J2.3 (Pin_3), J9.46 (Pin_46)
- new net PC13: J1.2 (Pin_2), J9.2 (Pin_2)
- new net PC14: J1.3 (Pin_3), J9.3 (Pin_3)
- new net PC15: J1.4 (Pin_4), J9.4 (Pin_4)
- new net PF0: J1.5 (Pin_5), J9.5 (Pin_5)
- new net PF1: J1.6 (Pin_6), J9.6 (Pin_6)
- new net PF6: J2.14 (Pin_14), J9.35 (Pin_35)
- new net PF7: J2.13 (Pin_13), J9.36 (Pin_36)
- new net VDDA: J1.9 (Pin_9), J9.9 (Pin_9)
Other:
- note added: "ADC from the analogue sensor"
- note added: "MEMORY"
- note added: "Microcontroller"
- note added: "PB6 is connected to the CLK line of the EEPROM"
- note added: "PB7 is connected to the SDA line on the EEPROM"
- note added: "The female connectors are used to represent the HAT"
- note added: "The male connectors are used to represent the microcontroller"
- note added: "This shows the EEPROM connection setup"
- note added: "This shows the microcontroller and its connections"
- moved on the sheet: U3, U4

Commit message: hail marry
Parts:
- J1, J2: footprint BAT60JFILM:SAMTEC_SSQ-120-03-G-D -> (none)
Changed lines of the file:
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@@
       (effects (font (size 1.27 1.27)) (justify left))
     )
-    (property "Footprint" "BAT60JFILM:SAMTEC_SSQ-120-03-G-D" (at 62.23 151.13 0)
+    (property "Footprint" "" (at 62.23 151.13 0)
       (effects (font (size 1.27 1.27)) hide)
     )
@@
       (effects (font (size 1.27 1.27)) (justify left))
     )
-    (property "Footprint" "BAT60JFILM:SAMTEC_SSQ-120-03-G-D" (at 77.47 151.13 0)
-      (effects (font (size 1.27 1.27)) hide)
-    )
+    (property "Footprint" "" (at 77.47 151.13 0)
+      (effects (font (size 1.27 1.27)) hide)
+    )

Commit message: the j's
Parts:
- removed U4: AT24CS01-STUM, Package_TO_SOT_SMD:SOT-23-5, symbol Memory_EEPROM:AT24CS01-STUM
- added U6: CAT24C256WI-GT3, BAT60JFILM:ON_Semi-751BD-01-12_2008-O-0, symbol best:CAT24C256WI-GT3
- J8: value Conn_01x02_Pin -> C5116481
Connections:
- net GND: now also U6.1 (A0), U6.2 (A1), U6.3 (A2), U6.4 (VSS), U6.7 (WP)
- net PB6: now also U6.6 (SCL)
- net PB7: now also U6.5 (SDA)
- net at C1.1, J8.1 (Pin_1): now also U6.8 (VCC)
Other:
- note removed: "Memory unit for debuging"
